File: Electronics/PCB (KiCAD)/RevB/LiBCM/LiBCM_BMS.sch (KiCad schematic (older format))
At the start: 437 parts, among them J12 Conn_01x02_Male, J13 Screw_Terminal_01x13, P3 BATT_CONN_12S, P4 BATT_CONN_18S, P5 BATT_CONN_18S, P6 BATT_CONN_12S, Q10 Q_PMOS_GSD, Q11 Q_PMOS_GSD, Q12 Q_PMOS_GSD, Q13 Q_PMOS_GSD, Q14 Q_PMOS_GSD, Q15 Q_PMOS_GSD, Q16 Q_PMOS_GSD, Q17 Q_PMOS_GSD, Q18 Q_PMOS_GSD, Q19 Q_PMOS_GSD, Q20 Q_NPN_BCEC, Q21 Q_PMOS_GSD, Q22 Q_PMOS_GSD, Q23 Q_PMOS_GSD, Q24 Q_PMOS_GSD, Q25 Q_PMOS_GSD, Q26 Q_PMOS_GSD, Q27 Q_PMOS_GSD, Q28 Q_PMOS_GSD, Q29 Q_PMOS_GSD, Q30 Q_PMOS_GSD, Q31 Q_PMOS_GSD, Q32 Q_PMOS_GSD, Q33 Q_NPN_BCEC, Q34 Q_PMOS_GSD, Q35 Q_PMOS_GSD, Q36 Q_PMOS_GSD, Q37 Q_PMOS_GSD, Q38 Q_PMOS_GSD, Q39 Q_PMOS_GSD, Q40 Q_PMOS_GSD, Q41 Q_PMOS_GSD, Q42 Q_PMOS_GSD, Q43 Q_PMOS_GSD, Q44 Q_PMOS_GSD, Q45 Q_PMOS_GSD, Q46 Q_NPN_BCEC, Q47 Q_PMOS_GSD, Q48 Q_PMOS_GSD, Q49 Q_PMOS_GSD, Q50 Q_PMOS_GSD, Q51 Q_PMOS_GSD, Q52 Q_PMOS_GSD, Q53 Q_PMOS_GSD, Q54 Q_PMOS_GSD, Q55 Q_PMOS_GSD, Q56 Q_PMOS_GSD, Q57 Q_PMOS_GSD, Q58 Q_PMOS_GSD, Q59 Q_NPN_BCEC, Q60 Q_PMOS_GSD, Q61 Q_PMOS_GSD, Q62 Q_PMOS_GSD, Q63 Q_PMOS_GSD, Q64 Q_PMOS_GSD, Q65 Q_PMOS_GSD, Q66 Q_PMOS_GSD, Q67 Q_PMOS_GSD, Q68 Q_PMOS_GSD, Q69 Q_PMOS_GSD, Q70 Q_PMOS_GSD, Q71 Q_PMOS_GSD, Q72 Q_NPN_BCEC, Q8 Q_PMOS_GSD, Q9 Q_PMOS_GSD, T1 Trans_7490100111, T2 Trans_7490100111, T3 Trans_7490100111, U10 LTC6820, U11 LTC6804-2, U12 LTC6804-2, U13 LTC6804-2, U14 LTC6804-2, U15 LTC6804-2

Commit message: RevB PCB Gerbers
Parts:
- removed J13: Screw_Terminal_01x13, Linsight:Conn_277-1232-ND, symbol Connector:Screw_Terminal_01x13
- removed P3, P6: BATT_CONN_12S, Linsight:CONN_HONDA-12S, symbol JTS_Parts:BATT_CONN_12S
- removed P4, P5: BATT_CONN_18S, Linsight:CONN_HONDA-18S, symbol JTS_Parts:BATT_CONN_18S
- added J13, J16: Conn_01x20, Connector_PinHeader_2.54mm:PinHeader_2x10_P2.54mm_Vertical, symbol Connector_Generic:Conn_01x20
- added J17, J18: Conn_01x14, Connector_PinHeader_2.54mm:PinHeader_2x07_P2.54mm_Vertical, symbol Connector_Generic:Conn_01x14
Connections:
- net C10pos: now also J13.11 (Pin_11)
- net C11pos: now also J13.12 (Pin_12)
- net CELL13pos: now also J13.14 (Pin_14)
- net CELL14pos: now also J13.15 (Pin_15)
- net CELL15pos: now also J13.16 (Pin_16)
- net CELL16pos: now also J13.17 (Pin_17)
- net CELL17pos: now also J13.18 (Pin_18)
- net CELL18pos: now also J13.19 (Pin_19), J16.1 (Pin_1)
- net CELL19pos: now also J16.2 (Pin_2)
- net CELL1pos: now also J13.2 (Pin_2)
- net CELL20pos: now also J16.3 (Pin_3)
- net CELL21pos: now also J16.4 (Pin_4)
- net CELL22pos: now also J16.5 (Pin_5)
- net CELL23pos: now also J16.6 (Pin_6)
- net CELL25pos: now also J16.8 (Pin_8)
- net CELL26pos: now also J16.9 (Pin_9)
- net CELL27pos: now also J16.10 (Pin_10)
- net CELL28pos: now also J16.11 (Pin_11)
- net CELL29pos: now also J16.12 (Pin_12)
- net CELL2pos: now also J13.3 (Pin_3)
- net CELL30pos: now also J16.13 (Pin_13)
- net CELL31pos: now also J16.14 (Pin_14)
- net CELL32pos: now also J16.15 (Pin_15)
- net CELL33pos: now also J16.16 (Pin_16)
- net CELL34pos: now also J16.17 (Pin_17)
- net CELL35pos: now also J16.18 (Pin_18)
- net CELL36pos: now also J16.19 (Pin_19)
- net CELL37pos: now also J17.2 (Pin_2)
- net CELL38pos: now also J17.3 (Pin_3)
- net CELL39pos: now also J17.4 (Pin_4)
- net CELL3pos: now also J13.4 (Pin_4)
- net CELL40pos: now also J17.5 (Pin_5)
- net CELL41pos: now also J17.6 (Pin_6)
- net CELL42pos: now also J17.7 (Pin_7)
- net CELL43pos: now also J17.8 (Pin_8)
- net CELL44pos: now also J17.9 (Pin_9)
- net CELL45pos: now also J17.10 (Pin_10)
- net CELL46pos: now also J17.11 (Pin_11)
- net CELL47pos: now also J17.12 (Pin_12)
- net CELL48pos: now also J17.13 (Pin_13)
- net CELL49pos: now also J18.2 (Pin_2)
- net CELL4pos: now also J13.5 (Pin_5)
- net CELL50pos: now also J18.3 (Pin_3)
- net CELL51pos: now also J18.4 (Pin_4)
- net CELL52pos: now also J18.5 (Pin_5)
- net CELL53pos: now also J18.6 (Pin_6)
- net CELL54pos: now also J18.7 (Pin_7)
- net CELL55pos: now also J18.8 (Pin_8)
- net CELL56pos: now also J18.9 (Pin_9)
- net CELL57pos: now also J18.10 (Pin_10)
- net CELL58pos: now also J18.11 (Pin_11)
- net CELL59pos: now also J18.12 (Pin_12)
- net CELL5pos: now also J13.6 (Pin_6)
- net CELL60pos: now also J18.13 (Pin_13)
- net CELL6pos: now also J13.7 (Pin_7)
- net CELL7pos: now also J13.8 (Pin_8)
- net CELL8pos: now also J13.9 (Pin_9)
- net CELL9pos: now also J13.10 (Pin_10)
- net GND_ISO_A: now also J13.1 (Pin_1)
- net GND_ISO_B: now also J13.13 (Pin_13)
- net GND_ISO_C: now also J16.7 (Pin_7)
- net GND_ISO_D: now also J17.1 (Pin_1)
- net GND_ISO_E: now also J18.1 (Pin_1)
- no-connect marks 32 -> 50
Other:
- note added: "42S"
- note added: "48S"
- note added: "C12+\nC11+\nC10+\nC09+\nC08+\nC07+\nC06+\nC05+\nC04+\nC03+\nC02+\nC01+\nC01-"
- note added: "C18+\nC17+\nC16+\nC15+\nC14+\nC13+\nC12+\nC11+\nC10+\nC09+\nC08+\nC07+\nC06+\nC05+\nC04+\nC03+\nC02+\nC01+\nC01-"
- note added: "FOR 42S CONFIGURATION:\n -LEAVE PINS C13+ TO C18+ \n DISCONNECTED"
- note removed: "CONNECT EITHER\nP3 (42S) OR P4 (48S)\nBUT NOT BOTH!!!!!!\n\nIN 42S CONFIGURATION\nCELLS 13 TO 18\nWILL RETURN 0 VOLTS\n"
- note removed: "Cell18+\nCell17+\nCell16+\nCell15+\nCell14+\nCell13+\nCell12+\nCell11+\nCell10+\nCell09+\nCell08+\nCell07+\nCell06+\nCell05+\nCell04+\nCell03+\nCell02+\nCell01+\nCell01-"
Changed lines of the file:
@@
 Text Label 2600 13300 0    60   ~ 0
 C0_A
-Text Notes 6250 6350 2    63   ~ 0
-Cell18+\nCell17+\nCell16+\nCell15+\nCell14+\nCell13+\nCell12+\nCell11+\nCell10+\nCell09+\nCell08+\nCell07+\nCell06+\nCell05+\nCell04+\nCell03+\nCell02+\nCell01+\nCell01-
+Text Notes 6000 6350 2    63   ~ 0
+C18+\nC17+\nC16+\nC15+\nC14+\nC13+\nC12+\nC11+\nC10+\nC09+\nC08+\nC07+\nC06+\nC05+\nC04+\nC03+\nC02+\nC01+\nC01-
 Text Label 8100 12950 0    60   ~ 0
 S1_B
@@
 	1    0    0    -1
 $EndComp
-Text Notes 16300 3150 2    63   ~ 0
+Text Notes 16400 3150 2    63   ~ 0
 Cell48+\nCell47+\nCell46+\nCell45+\nCell44+\nCell43+\nCell42+\nCell41+\nCell40+\nCell39+\nCell38+\nCell37+\nCell37-\n
 Text Label 19200 12950 0    60   ~ 0
@@
 Text Label 13650 12950 0    60   ~ 0
 S1_C
-Text Notes 10450 3750 2    63   ~ 0
+Text Notes 10550 3750 2    63   ~ 0
 Cell36+\nCell35+\nCell34+\nCell33+\nCell32+\nCell31+\nCell30+\nCell29+\nCell28+\nCell27+\nCell26+\nCell25+\nCell25-(24+)\nCell23+\nCell22+\nCell21+\nCell20+\nCell19+\nCell19-(18+)
 $Comp
@@
 Wire Wire Line
 	4150 9200 3850 9200
-$Comp
-L JTS_Parts:BATT_CONN_12S P6
-U 1 1 6E989E63
-P 16600 2100
-F 0 "P6" H 16750 950 118 0000 C CNN
-F 1 "BATT_CONN_12S" H 16692 3285 118 0000 C CNN
-F 2 "Linsight:CONN_HONDA-12S" H 16400 1050 118 0001 C CNN
-F 3 "" H 16400 1050 118 0001 C CNN
-	1    16600 2100
-	-1   0    0    -1
-$EndComp
 Text Notes 12200 1150 0    118  ~ 0
 BATTERY BAY 2: 18S MODULE\n(MIDDLE BAY)\nHIGHEST 12 CELLS
-$Comp
-L JTS_Parts:BATT_CONN_18S P5
-U 1 1 60BC1114
-P 10750 2700
-F 0 "P5" H 10900 1550 118 0000 C CNN
-F 1 "BATT_CONN_18S" H 10842 4685 118 0000 C CNN
-F 2 "Linsight:CONN_HONDA-18S" H 10550 1650 118 0001 C CNN
-F 3 "" H 10550 1650 118 0001 C CNN
-	1    10750 2700
-	-1   0    0    -1
-$EndComp
 Wire Wire Line
 	9350 1750 9350 9200
@@
 Wire Wire Line
 	6150 11400 6150 6950
-$Comp
-L JTS_Parts:BATT_CONN_18S P4
-U 1 1 631124E8
-P 5550 5300
-F 0 "P4" H 5700 4150 118 0000 C CNN
-F 1 "BATT_CONN_18S" V 5700 7900 118 0000 C CNN
-F 2 "Linsight:CONN_HONDA-18S" H 5350 4250 118 0001 C CNN
-F 3 "" H 5350 4250 118 0001 C CNN
-	1    5550 5300
-	1    0    0    -1
-$EndComp
-$Comp
-L JTS_Parts:BATT_CONN_12S P3
-U 1 1 63114474
-P 4250 5300
-F 0 "P3" H 4400 4150 118 0000 C CNN
-F 1 "BATT_CONN_12S" V 4400 7100 118 0000 C CNN
-F 2 "Linsight:CONN_HONDA-12S" H 4050 4250 118 0001 C CNN
-F 3 "" H 4050 4250 118 0001 C CNN
-	1    4250 5300
-	-1   0    0    -1
-$EndComp
 Wire Wire Line
 	4400 1600 4400 5100
@@
 Wire Wire Line
 	6350 1350 6350 6750
-Text Notes 3950 8300 0    110  ~ 0
-CONNECT EITHER\nP3 (42S) OR P4 (48S)\nBUT NOT BOTH!!!!!!\n\nIN 42S CONFIGURATION\nCELLS 13 TO 18\nWILL RETURN 0 VOLTS\n
+Text Notes 4050 7600 0    79   ~ 0
+FOR 42S CONFIGURATION:\n -LEAVE PINS C13+ TO C18+ \n  DISCONNECTED
 Text Notes 9450 5200 0    110  ~ 0
 U11/U12/U13 ARE NOT\nGALVANICALLY ISOLATED\nFROM EACH OTHER\n(BUT U14 IS)
@@
 	1    0    0    -1
 $EndComp
-$Comp
-L Connector:Screw_Terminal_01x13 J13
-U 1 1 672F40D1
-P 22200 2500
-F 0 "J13" H 22118 1675 50  0000 C CNN
-F 1 "Screw_Terminal_01x13" H 22118 1766 50  0000 C CNN
-F 2 "Linsight:Conn_277-1232-ND" H 22200 2500 50  0001 C CNN
-F 3 "~" H 22200 2500 50  0001 C CNN
-	1    22200 2500
-	-1   0    0    1
-$EndComp
 Wire Wire Line
 	21600 10550 21600 10750
@@
 	6150 15300 5750 15300
 Connection ~ 5750 15300
+$Comp
+L Connector_Generic:Conn_01x20 J13
+U 1 1 60FD5054
+P 5650 5400
+F 0 "J13" H 5568 4175 50  0000 C CNN
+F 1 "Conn_01x20" H 5568 4266 50  0000 C CNN
+F 2 "Connector_PinHeader_2.54mm:PinHeader_2x10_P2.54mm_Vertical" H 5650 5400 50  0001 C CNN
+F 3 "~" H 5650 5400 50  0001 C CNN
+	1    5650 5400
+	1    0    0    1
+$EndComp
+$Comp
+L Connector_Generic:Conn_01x20 J16
+U 1 1 60FDCF82
+P 10650 2800
+F 0 "J16" H 10568 1575 50  0000 C CNN
+F 1 "Conn_01x20" H 10568 1666 50  0000 C CNN
+F 2 "Connector_PinHeader_2.54mm:PinHeader_2x10_P2.54mm_Vertical" H 10650 2800 50  0001 C CNN
+F 3 "~" H 10650 2800 50  0001 C CNN
+	1    10650 2800
+	-1   0    0    1
+$EndComp
+$Comp
+L Connector_Generic:Conn_01x14 J17
+U 1 1 60FECDD3
+P 16500 2500
+F 0 "J17" H 16418 1575 50  0000 C CNN
+F 1 "Conn_01x14" H 16418 1666 50  0000 C CNN
+F 2 "Connector_PinHeader_2.54mm:PinHeader_2x07_P2.54mm_Vertical" H 16500 2500 50  0001 C CNN
+F 3 "~" H 16500 2500 50  0001 C CNN
+	1    16500 2500
+	-1   0    0    1
+$EndComp
+$Comp
+L Connector_Generic:Conn_01x14 J18
+U 1 1 60FF4D07
+P 22200 2500
+F 0 "J18" H 22118 1575 50  0000 C CNN
+F 1 "Conn_01x14" H 22118 1666 50  0000 C CNN
+F 2 "Connector_PinHeader_2.54mm:PinHeader_2x07_P2.54mm_Vertical" H 22200 2500 50  0001 C CNN
+F 3 "~" H 22200 2500 50  0001 C CNN
+	1    22200 2500
+	-1   0    0    1
+$EndComp
+NoConn ~ 22400 1800
+NoConn ~ 16700 1800
+NoConn ~ 10850 1800
+NoConn ~ 5450 4400
+NoConn ~ 5700 3300
+Text Notes 4300 6350 2    63   ~ 0
+C12+\nC11+\nC10+\nC09+\nC08+\nC07+\nC06+\nC05+\nC04+\nC03+\nC02+\nC01+\nC01-
+Text Notes 4250 4950 2    110  ~ 0
+42S
+Text Notes 6050 4150 2    110  ~ 0
+48S
+NoConn ~ 4350 6300
+NoConn ~ 4350 6200
+NoConn ~ 4350 6100
+NoConn ~ 4350 6000
+NoConn ~ 4350 5900
+NoConn ~ 4350 5700
+NoConn ~ 4350 5800
+NoConn ~ 4350 5600
+NoConn ~ 4350 5500
+NoConn ~ 4350 5400
+NoConn ~ 4350 5300
+NoConn ~ 4350 5200
+NoConn ~ 4350 5100
 $EndSCHEMATC
