File: Electronics/PCB (KiCAD)/RevB/LiBCM/LiBCM.kicad_pcb (KiCad board)
At the start: 4 copper layers, 355 x 160 mm, 624 parts, among them J1 Conn_01x08, J10 Screw_Terminal_01x03, J11 Screw_Terminal_01x08, J12 Conn_01x02_Male, J13 Screw_Terminal_01x13, J14 Conn_01x04, J15 Conn_01x02, J2 Conn_01x08, J3 Conn_01x08, J4 Conn_02x03_Odd_Even, J5 Conn_01x08, J6 Conn_01x08, J7 Conn_01x08, J8 Screw_Terminal_01x06, J9 Screw_Terminal_01x08, M1 Fan, M2 Fan, M3 Fan, P1 OEM_BCM_Connector, P2 Conn_WallPlug_Earth, P3 BATT_CONN_12S, P4 BATT_CONN_18S, P5 BATT_CONN_18S, P6 BATT_CONN_12S, Q1 Q_NMOS_GSD, Q10 Q_PMOS_GSD, Q11 Q_PMOS_GSD, Q12 Q_PMOS_GSD, Q13 Q_PMOS_GSD, Q14 Q_PMOS_GSD, Q15 Q_PMOS_GSD, Q16 Q_PMOS_GSD, Q17 Q_PMOS_GSD, Q18 Q_PMOS_GSD, Q19 Q_PMOS_GSD, Q2 Q_NMOS_GSD, Q20 Q_NPN_BCEC, Q21 Q_PMOS_GSD, Q22 Q_PMOS_GSD, Q23 Q_PMOS_GSD, Q24 Q_PMOS_GSD, Q25 Q_PMOS_GSD, Q26 Q_PMOS_GSD, Q27 Q_PMOS_GSD, Q28 Q_PMOS_GSD, Q29 Q_PMOS_GSD, Q3 Q_NMOS_GSD, Q30 Q_PMOS_GSD, Q31 Q_PMOS_GSD, Q32 Q_PMOS_GSD, Q33 Q_NPN_BCEC, Q34 Q_PMOS_GSD, Q35 Q_PMOS_GSD, Q36 Q_PMOS_GSD, Q37 Q_PMOS_GSD, Q38 Q_PMOS_GSD, Q39 Q_PMOS_GSD, Q4 Q_NMOS_GSD, Q40 Q_PMOS_GSD, Q41 Q_PMOS_GSD, Q42 Q_PMOS_GSD, Q43 Q_PMOS_GSD, Q44 Q_PMOS_GSD, Q45 Q_PMOS_GSD, Q46 Q_NPN_BCEC, Q47 Q_PMOS_GSD, Q48 Q_PMOS_GSD, Q49 Q_PMOS_GSD, Q5 Q_NMOS_GSD, Q50 Q_PMOS_GSD, Q51 Q_PMOS_GSD, Q52 Q_PMOS_GSD, Q53 Q_PMOS_GSD, Q54 Q_PMOS_GSD, Q55 Q_PMOS_GSD, Q56 Q_PMOS_GSD, Q57 Q_PMOS_GSD, Q58 Q_PMOS_GSD, Q59 Q_NPN_BCEC, Q6 Q_NMOS_GSD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

Commit message: RevB PCB Gerbers
Parts:
- removed P3, P6: BATT_CONN_12S, Linsight:CONN_HONDA-12S
- removed P4, P5: BATT_CONN_18S, Linsight:CONN_HONDA-18S
- added J16: Conn_01x20, Connector_PinHeader_2.54mm:PinHeader_2x10_P2.54mm_Vertical, B.Cu at (179.2, 118.2)
- added J17: Conn_01x14, Connector_PinHeader_2.54mm:PinHeader_2x07_P2.54mm_Vertical, B.Cu at (275.0, 115.0)
- added J18: Conn_01x14, Connector_PinHeader_2.54mm:PinHeader_2x07_P2.54mm_Vertical, B.Cu at (227.0, 138.8)
- added REF**: OSHW-Logo_11.4x12mm_SilkScreen, Symbol:OSHW-Logo_11.4x12mm_SilkScreen, F.Cu at (373.0, 186.8)
- J13: value Screw_Terminal_01x13 -> Conn_01x20; footprint Linsight:Conn_277-1232-ND -> Connector_PinHeader_2.54mm:PinHeader_2x10_P2.54mm_Vertical; moved to B.Cu
- J9: moved to B.Cu
- moved J13 180.6 mm to (38.5, 80.0), turned to 180 degrees
- moved R94 56.2 mm to (98.8, 40.5), turned to 0 degrees
- moved TH1 52.1 mm to (103.5, 40.5), turned to 270 degrees
- moved R93 51.3 mm to (98.8, 44.5), turned to 0 degrees
- moved Q19 50.9 mm to (92.8, 40.5), turned to 0 degrees
- moved R119 48.7 mm to (89.0, 40.0), turned to 0 degrees
- moved Q18 45.6 mm to (92.8, 44.5), turned to 0 degrees
- moved R118 45.4 mm to (89.0, 43.2), turned to 0 degrees
- moved R92 31.5 mm to (83.2, 43.5), turned to 0 degrees
- moved C41 27.4 mm to (64.0, 40.0), turned to 180 degrees
- moved R107 25.8 mm to (59.8, 40.0), turned to 180 degrees
- moved Q17 25.3 mm to (77.2, 43.5), turned to 0 degrees
- moved R117 24.7 mm to (73.0, 42.8), turned to 0 degrees
- moved C47 15.5 mm to (59.8, 42.5), turned to 180 degrees
- moved D1 8.95 mm to (166.0, 121.2)
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Connections:
- H4 pad 1: Net-(H4-Pad1) -> (no net)
- H6 pad 1: Net-(H6-Pad1) -> (no net)
- J1 pad 1: Net-(J1-Pad1) -> (no net)
- J1 pad 2: Net-(J1-Pad2) -> (no net)
- J1 pad 4: Net-(J1-Pad4) -> (no net)
- J1 pad 8: Net-(J1-Pad8) -> (no net)
- J13 pad 1: GND_ISO_E -> GND_ISO_A
- J13 pad 10: /LiBCM BMS/CELL57pos -> /LiBCM BMS/CELL9pos
- J13 pad 11: /LiBCM BMS/CELL58pos -> /LiBCM BMS/C10pos
- J13 pad 12: /LiBCM BMS/CELL59pos -> /LiBCM BMS/C11pos
- J13 pad 13: /LiBCM BMS/CELL60pos -> GND_ISO_B
- J13 pad 2: /LiBCM BMS/CELL49pos -> /LiBCM BMS/CELL1pos
- J13 pad 3: /LiBCM BMS/CELL50pos -> /LiBCM BMS/CELL2pos
- J13 pad 4: /LiBCM BMS/CELL51pos -> /LiBCM BMS/CELL3pos
- J13 pad 5: /LiBCM BMS/CELL52pos -> /LiBCM BMS/CELL4pos
- J13 pad 6: /LiBCM BMS/CELL53pos -> /LiBCM BMS/CELL5pos
- J13 pad 7: /LiBCM BMS/CELL54pos -> /LiBCM BMS/CELL6pos
- J13 pad 8: /LiBCM BMS/CELL55pos -> /LiBCM BMS/CELL7pos
- J13 pad 9: /LiBCM BMS/CELL56pos -> /LiBCM BMS/CELL8pos
- J6 pad 1: Net-(J6-Pad1) -> (no net)
- J6 pad 2: Net-(J6-Pad2) -> (no net)
- P1 pad A05: Net-(P1-PadA05) -> (no net)
- P1 pad A06: Net-(P1-PadA06) -> (no net)
- P1 pad A09: Net-(P1-PadA09) -> (no net)
- P1 pad A10: Net-(P1-PadA10) -> (no net)
- P1 pad A17: Net-(P1-PadA17) -> (no net)
- P1 pad A18: Net-(P1-PadA18) -> (no net)
- P1 pad A19: Net-(P1-PadA19) -> (no net)
- P1 pad A22: Net-(P1-PadA22) -> (no net)
- P1 pad A23: Net-(P1-PadA23) -> (no net)
- P1 pad A26: Net-(P1-PadA26) -> (no net)
- P1 pad B06: Net-(P1-PadB06) -> (no net)
- P1 pad B07: Net-(P1-PadB07) -> (no net)
- P1 pad B10: Net-(P1-PadB10) -> (no net)
- P1 pad B13: Net-(P1-PadB13) -> (no net)
- P1 pad B14: Net-(P1-PadB14) -> (no net)
- P1 pad B15: Net-(P1-PadB15) -> (no net)
- P1 pad B16: Net-(P1-PadB16) -> (no net)
- P1 pad B17: Net-(P1-PadB17) -> (no net)
- P1 pad B18: Net-(P1-PadB18) -> (no net)
- P1 pad B21: Net-(P1-PadB21) -> (no net)
- T1 pad 12: Net-(T1-Pad12) -> (no net)
- T1 pad 13: Net-(T1-Pad13) -> (no net)
- T1 pad 4: Net-(T1-Pad4) -> (no net)
- T1 pad 5: Net-(T1-Pad5) -> (no net)
- T2 pad 12: Net-(T2-Pad12) -> (no net)
- T2 pad 13: Net-(T2-Pad13) -> (no net)
- T2 pad 4: Net-(T2-Pad4) -> (no net)
- T2 pad 5: Net-(T2-Pad5) -> (no net)
- T3 pad 12: Net-(T3-Pad12) -> (no net)
- T3 pad 13: Net-(T3-Pad13) -> (no net)
- T3 pad 4: Net-(T3-Pad4) -> (no net)
- T3 pad 5: Net-(T3-Pad5) -> (no net)
- U11 pad 28: Net-(U11-Pad28) -> (no net)
- U11 pad 29: Net-(U11-Pad29) -> (no net)
- U11 pad 32: Net-(U11-Pad32) -> (no net)
- U11 pad 33: Net-(U11-Pad33) -> (no net)
- U12 pad 28: Net-(U12-Pad28) -> (no net)
- U12 pad 29: Net-(U12-Pad29) -> (no net)
- U12 pad 32: Net-(U12-Pad32) -> (no net)
- U12 pad 33: Net-(U12-Pad33) -> (no net)
- U13 pad 28: Net-(U13-Pad28) -> (no net)
- U13 pad 29: Net-(U13-Pad29) -> (no net)
- U13 pad 32: Net-(U13-Pad32) -> (no net)
- U13 pad 33: Net-(U13-Pad33) -> (no net)
- U14 pad 28: Net-(U14-Pad28) -> (no net)
- U14 pad 29: Net-(U14-Pad29) -> (no net)
- U14 pad 32: Net-(U14-Pad32) -> (no net)
- U14 pad 33: Net-(U14-Pad33) -> (no net)
- U15 pad 28: Net-(U15-Pad28) -> (no net)
- U15 pad 29: Net-(U15-Pad29) -> (no net)
- U15 pad 32: Net-(U15-Pad32) -> (no net)
- U15 pad 33: Net-(U15-Pad33) -> (no net)
- U5 pad 3: Net-(U5-Pad3) -> (no net)
- U5 pad 5: Net-(U5-Pad5) -> (no net)
- U8 pad 11: Net-(U8-Pad11) -> (no net)
- U8 pad 14: Net-(U8-Pad14) -> (no net)
- U8 pad 4: Net-(U8-Pad4) -> (no net)
- U8 pad 6: Net-(U8-Pad6) -> (no net)
- U8 pad 8: Net-(U8-Pad8) -> (no net)
- U8 pad 9: Net-(U8-Pad9) -> (no net)
- U9 pad 3: Net-(U9-Pad3) -> (no net)
Routing:
- net GND_ISO_B: track 260.5 -> 372.0 mm
- net /LiBCM BMS/CELL14pos: track 182.2 -> 77.8 mm, vias 1 -> 2
- net GND_ENG: track 3657.3 -> 3555.4 mm, vias 743 -> 697
- net /LiBCM BMS/CELL16pos: track 164.9 -> 67.4 mm, vias 3 -> 2
- net /LiBCM BMS/CELL18pos: track 315.8 -> 218.7 mm, vias 2 -> 3
- net GND_ISO_C: track 496.9 -> 576.3 mm
- net /LiBCM BMS/CELL17pos: track 132.8 -> 67.9 mm, vias 3 -> 0
- net /LiBCM BMS/CELL1pos: track 200.5 -> 139.3 mm
- net /LiBCM BMS/CELL15pos: track 140.1 -> 79.7 mm, vias 1 -> 2
- net /LiBCM BMS/T_A: track 15.6 -> 72.5 mm, vias 2 -> 0
- net /LiBCM BMS/CELL13pos: track 146.4 -> 90.6 mm, vias 1 -> 2
- net /LiBCM BMS/S1_A: track 3.42 -> 50.8 mm, vias 0 -> 2
- net GND_ISO_D: track 275.6 -> 316.5 mm, vias 8 -> 6
- net /LiBCM BMS/CELL3pos: track 181.0 -> 141.0 mm, vias 3 -> 0
- net /LiBCM BMS/S2_A: track 7.43 -> 47.3 mm
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- added copper zone on B.Cu, net (none)
- added copper zone on F.Cu, net (none)
- added copper zone on F.Cu, net /GRID_SENSE_L2
- added copper zone on F.Cu, net /L1_GRID
- added copper zone on F.Cu, net /TRIAC_GATE
- added copper zone on B.Cu, net GND_ISO_A
- removed copper zone on B.Cu, net /LiBCM BMS/CELL20pos
- removed copper zone on B.Cu, net /LiBCM BMS/CELL2pos
- removed copper zone on B.Cu, net /LiBCM BMS/CELL4pos
Other:
- rule via_min_size: 0.4 -> 0.59
- board text added: "1+ 3+ 5+ 7+ 9+ 11+ 13+ 15+ 17+ NC"
- board text added: "1- 2+ 4+ 6+ 8+ 10+ 12+ 14+ 16+ 18+"
- board text added: "12V F+ F+ F+ F- F- F- GND"
- board text added: "36+ 34+ 32+ 30+ 28+ 26+ 24+ 22+ 20+ 19-"
- board text added: "48+ 46+ 44+ 42+ 40+ 38+ 37-"
- board text added: "54S IMA BATTERY: SHORT 60+ TO 54+ SHORT 49- TO 48+ LITHIUM 12V BATTERY: SHORT 60+ TO 52+ LEAVE 49- FLOATING!"
- board text added: "60+ 58+ 56+ 54+ 52+ 50+ 49-"
- board text added: "CONNECTING J11/J13/J16/J17/J18 INCORRECTLY WILL DAMAGE TRACES/COMPONENTS ON THIS PCB."
- board text added: "FAILURE TO FOLLOW THESE RULES WILL DESTROY IC U12: DO NOT PLACE FUSE/SWITCH BETWEEN CELLS C1:C36!!!!! CONNECT CELLS C1:C36 TOGETHER WITH HIGH CURRENT CABLES BEFORE CONNECTING J13/J16 DISCONNECT J13/J16 BEFORE REMOVING HIGH CURRENT CABLES BETWEEN C1:C36"
- board text added: "HAZARDOUS VOLTAGE PRESENT EVEN"
- board text added: "J13"
- board text added: "J16"
- board text added: "J17"
- board text added: "J18"
- board text added: "J9"
- board text added: "NC 35+ 33+ 31+ 29+ 27+ 25+ 23+ 21+ 19+"
- board text added: "NC 47+ 45+ 43+ 41+ 39+ 37+"
- board text added: "NC 59+ 57+ 55+ 53+ 51+ 49+"
- board text added: "PLACE FUSE & SWITCH BETWEEN C36+ & C37-"
- board text added: "THIS SECTION GALVANICALLY ISOLATED FROM ALL OTHER SECTIONS"
- board text added: "THIS SECTION IS: -HIGH VOLTAGE WHEN CONN J18 IS CONNECTED TO IMA -TOUCH SAFE WHEN J18 IS UNPLUGGED OR LOW VOLTAGE"
- board text added: "TO USE LiDisplay: -J14: CONNECT CABLE -J15: REMOVE JUMPER TO USE HLINE: -J14: SHORT TX & RX -J15: SHORT PINS -P1: CONNECT HLINE TO BCM CONN B01"
- board text added: "UNDER HVDCDC:"
- board text added: "WHEN IMA SWITCH IS OFF"
- board text removed: "1- 1+"
- board text removed: "12 F+ F+ F+ F- F- F-"
- board text removed: "19- 19+"
- board text removed: "49- 49+ 50+ 51+ 52+ 53+ 54+ 55+ 56+ 57+ 58+ 59+ 60+"
- board text removed: "AUX BATT"
- board text removed: "CONNECTING P3/P4/P5/P6/J11 INCORRECTLY COULD DAMAGE TRACES/COMPONENTS ON THIS PCB."
- board text removed: "DANGER!!! HIGH VOLTAGE!!!"
- board text removed: "GND"
- board text removed: "NC NC"
- board text removed: "NC NC NC 12+ 10+ 8+ 6+ 4+ 2+ 1-"
- board text removed: "NC NC NC 18+ 16+ 14+ 12+ 10+ 8+ 6+ 4+ 2+"
- board text removed: "NC NC NC 36+ 34+ 32+ 30+ 28+ 26+ 24+ 22+ 20+"
- board text removed: "NC NC NC 48+ 46+ 44+ 42+ 40+ 38+ 37-"
- board text removed: "NC NC NC NC 11+ 9+ 7+ 5+ 3+ 1+"
- board text removed: "NC NC NC NC 17+ 15+ 13+ 11+ 9+ 7+ 5+ 3+"
- board text removed: "NC NC NC NC 35+ 33+ 31+ 29+ 27+ 25+ 23+ 21+"
- board text removed: "NC NC NC NC 47+ 45+ 43+ 41+ 39+ 37+"
- board text removed: "ONLY ONE"
- board text removed: "P3"
- board text removed: "P4"
- board text removed: "P5"
- board text removed: "P6"
- board text removed: "PLACE FUSE/SWITCH BETWEEN C36+ & C37-"
- board text removed: "TAB"
- board text removed: "TO USE LiDisplay: -J14: CONNECT CABLE -J15: REMOVE JUMPER TO USE HLINE: -J14: SHORT TX & RX -J15: SHORT PINS -P1: CONNECT HLINE TO B01"
- board text removed: "USB"
- board text removed: "USE"
- board text removed: "YOU MUST CONNECT CELLS C1:C36 TOGETHER WITH HIGH CURRENT CABLES BEFORE CONNECTING P3/P4/P5 YOU MUST DISCONNECT P3/P4/P5 BEFORE REMOVING HIGH CURRENT CABLES BETWEEN C1:C36 DO NOT PLACE FUSE/SWITCH BETWEEN CELLS C1:C36!!!!! FAILURE TO FOLLOW THESE RULES WILL DESTROY IC U12!"

Commit message: Final BOM prep prior to RevB Assembly
Parts:
- C152, C31: value 22n -> 68n
- R69, R72: value 10k -> 10k@0.25W
- R70, R71: value 71k5 -> 20k@0.5W
Connections:
- H4 pad 1: (no net) -> Net-(H4-Pad1)
- H6 pad 1: (no net) -> Net-(H6-Pad1)
- J1 pad 1: (no net) -> Net-(J1-Pad1)
- J1 pad 2: (no net) -> Net-(J1-Pad2)
- J1 pad 4: (no net) -> Net-(J1-Pad4)
- J1 pad 8: (no net) -> Net-(J1-Pad8)
- J13 pad 20: (no net) -> Net-(J13-Pad20)
- J16 pad 20: (no net) -> Net-(J16-Pad20)
- J17 pad 14: (no net) -> Net-(J17-Pad14)
- J18 pad 14: (no net) -> Net-(J18-Pad14)
- J6 pad 1: (no net) -> Net-(J6-Pad1)
- J6 pad 2: (no net) -> Net-(J6-Pad2)
- P1 pad A05: (no net) -> Net-(P1-PadA05)
- P1 pad A06: (no net) -> Net-(P1-PadA06)
- P1 pad A09: (no net) -> Net-(P1-PadA09)
- P1 pad A10: (no net) -> Net-(P1-PadA10)
- P1 pad A17: (no net) -> Net-(P1-PadA17)
- P1 pad A18: (no net) -> Net-(P1-PadA18)
- P1 pad A19: (no net) -> Net-(P1-PadA19)
- P1 pad A22: (no net) -> Net-(P1-PadA22)
- P1 pad A23: (no net) -> Net-(P1-PadA23)
- P1 pad A26: (no net) -> Net-(P1-PadA26)
- P1 pad B06: (no net) -> Net-(P1-PadB06)
- P1 pad B07: (no net) -> Net-(P1-PadB07)
- P1 pad B10: (no net) -> Net-(P1-PadB10)
- P1 pad B13: (no net) -> Net-(P1-PadB13)
- P1 pad B14: (no net) -> Net-(P1-PadB14)
- P1 pad B15: (no net) -> Net-(P1-PadB15)
- P1 pad B16: (no net) -> Net-(P1-PadB16)
- P1 pad B17: (no net) -> Net-(P1-PadB17)
- P1 pad B18: (no net) -> Net-(P1-PadB18)
- P1 pad B21: (no net) -> Net-(P1-PadB21)
- T1 pad 12: (no net) -> Net-(T1-Pad12)
- T1 pad 13: (no net) -> Net-(T1-Pad13)
- T1 pad 4: (no net) -> Net-(T1-Pad4)
- T1 pad 5: (no net) -> Net-(T1-Pad5)
- T2 pad 12: (no net) -> Net-(T2-Pad12)
- T2 pad 13: (no net) -> Net-(T2-Pad13)
- T2 pad 4: (no net) -> Net-(T2-Pad4)
- T2 pad 5: (no net) -> Net-(T2-Pad5)
- T3 pad 12: (no net) -> Net-(T3-Pad12)
- T3 pad 13: (no net) -> Net-(T3-Pad13)
- T3 pad 4: (no net) -> Net-(T3-Pad4)
- T3 pad 5: (no net) -> Net-(T3-Pad5)
- U11 pad 28: (no net) -> Net-(U11-Pad28)
- U11 pad 29: (no net) -> Net-(U11-Pad29)
- U11 pad 32: (no net) -> Net-(U11-Pad32)
- U11 pad 33: (no net) -> Net-(U11-Pad33)
- U12 pad 28: (no net) -> Net-(U12-Pad28)
- U12 pad 29: (no net) -> Net-(U12-Pad29)
- U12 pad 32: (no net) -> Net-(U12-Pad32)
- U12 pad 33: (no net) -> Net-(U12-Pad33)
- U13 pad 28: (no net) -> Net-(U13-Pad28)
- U13 pad 29: (no net) -> Net-(U13-Pad29)
- U13 pad 32: (no net) -> Net-(U13-Pad32)
- U13 pad 33: (no net) -> Net-(U13-Pad33)
- U14 pad 28: (no net) -> Net-(U14-Pad28)
- U14 pad 29: (no net) -> Net-(U14-Pad29)
- U14 pad 32: (no net) -> Net-(U14-Pad32)
- U14 pad 33: (no net) -> Net-(U14-Pad33)
- U15 pad 28: (no net) -> Net-(U15-Pad28)
- U15 pad 29: (no net) -> Net-(U15-Pad29)
- U15 pad 32: (no net) -> Net-(U15-Pad32)
- U15 pad 33: (no net) -> Net-(U15-Pad33)
- U5 pad 3: (no net) -> Net-(U5-Pad3)
- U5 pad 5: (no net) -> Net-(U5-Pad5)
- U8 pad 11: (no net) -> Net-(U8-Pad11)
- U8 pad 14: (no net) -> Net-(U8-Pad14)
- U8 pad 4: (no net) -> Net-(U8-Pad4)
- U8 pad 6: (no net) -> Net-(U8-Pad6)
- U8 pad 8: (no net) -> Net-(U8-Pad8)
- U8 pad 9: (no net) -> Net-(U8-Pad9)
- U9 pad 3: (no net) -> Net-(U9-Pad3)
