File: Electronics/PCB (KiCAD)/RevC/KiCAD/LiBCM_BMS.sch (KiCad schematic (older format))
At the start: 457 parts, among them J13 Conn_01x20, J16 Conn_01x20, J17 Conn_01x14, J18 Conn_01x14, Q10 Q_PMOS_GSD, Q11 Q_PMOS_GSD, Q12 Q_PMOS_GSD, Q13 Q_PMOS_GSD, Q14 Q_PMOS_GSD, Q15 Q_PMOS_GSD, Q16 Q_PMOS_GSD, Q17 Q_PMOS_GSD, Q18 Q_PMOS_GSD, Q19 Q_PMOS_GSD, Q20 Q_NPN_BCEC, Q21 Q_PMOS_GSD, Q22 Q_PMOS_GSD, Q23 Q_PMOS_GSD, Q24 Q_PMOS_GSD, Q25 Q_PMOS_GSD, Q26 Q_PMOS_GSD, Q27 Q_PMOS_GSD, Q28 Q_PMOS_GSD, Q29 Q_PMOS_GSD, Q30 Q_PMOS_GSD, Q31 Q_PMOS_GSD, Q32 Q_PMOS_GSD, Q33 Q_NPN_BCEC, Q34 Q_PMOS_GSD, Q35 Q_PMOS_GSD, Q36 Q_PMOS_GSD, Q37 Q_PMOS_GSD, Q38 Q_PMOS_GSD, Q39 Q_PMOS_GSD, Q40 Q_PMOS_GSD, Q41 Q_PMOS_GSD, Q42 Q_PMOS_GSD, Q43 Q_PMOS_GSD, Q44 Q_PMOS_GSD, Q45 Q_PMOS_GSD, Q46 Q_NPN_BCEC, Q47 Q_PMOS_GSD, Q48 Q_PMOS_GSD, Q49 Q_PMOS_GSD, Q50 Q_PMOS_GSD, Q51 Q_PMOS_GSD, Q52 Q_PMOS_GSD, Q53 Q_PMOS_GSD, Q54 Q_PMOS_GSD, Q55 Q_PMOS_GSD, Q56 Q_PMOS_GSD, Q57 Q_PMOS_GSD, Q58 Q_PMOS_GSD, Q59 Q_NPN_BCEC, Q60 Q_PMOS_GSD, Q61 Q_PMOS_GSD, Q62 Q_PMOS_GSD, Q63 Q_PMOS_GSD, Q64 Q_PMOS_GSD, Q65 Q_PMOS_GSD, Q66 Q_PMOS_GSD, Q67 Q_PMOS_GSD, Q68 Q_PMOS_GSD, Q69 Q_PMOS_GSD, Q70 Q_PMOS_GSD, Q71 Q_PMOS_GSD, Q72 Q_NPN_BCEC, Q8 Q_PMOS_GSD, Q9 Q_PMOS_GSD, T1 Trans_7490100111, T2 Trans_7490100111, T3 Trans_7490100111, U10 LTC6820, U11 LTC6804-2, U12 LTC6804-2, U13 LTC6804-2, U14 LTC6804-2, U15 LTC6804-2

Commit message: Schematic complete
Still considering adding a few items, but probably done.
Parts:
- removed R81: 1k24, Resistor_SMD:R_0805_2012Metric, symbol LiBCM-rescue:R
- removed R82: 7k32, Resistor_SMD:R_0805_2012Metric, symbol LiBCM-rescue:R
- gave numbers to parts that had none: 26
Other:
- note added: "BATTERY BAY 1: 12S MODULE\n(CLOSEST TO JUNCTION BOARD)"
- note added: "BATTERY BAY 2 (MIDDLE BAY): 18S MODULE"
- note added: "BATTERY BAY 3 (FURTHEST FROM JUNCTION BOARD): 18S"
- note added: "CELL18pos connects to both\nJ13 & J16. Thus, a small portion\nof assist/regen current flows\nthru this trace. This causes about\n1 mV error per regen/assist amp.\nExamples:\n+052A regen causes +50mV reading\n-129A assist causes -90mV reading\n \nLTC6813 would prevent this."
- note added: "CELL24pos doesn't have the same issue\nas CELL18pos (see note), because C24+\nconnects between QTY2 LTC6804 ICs,\nwhereas C18+ connects between QTY2\nBMS sense connectors (hence no current)"
- note removed: "BATTERY BAY 1: 12S MODULE\n(CLOSEST TO JUNCTION BOARD)\nALL 12 CELLS"
- note removed: "BATTERY BAY 2: 18S MODULE\n(MIDDLE BAY)\nHIGHEST 12 CELLS"
- note removed: "BATTERY BAY 3: 18S"
- moved on the sheet: J13

Commit message: RevC PCB in Layout
Parts:
- removed C176: DNP, Capacitor_SMD:C_0805_2012Metric, symbol LiBCM-rescue:C
- removed R351: DNP, Resistor_SMD:R_0805_2012Metric, symbol LiBCM-rescue:R
- added R359: 20, Resistor_SMD:R_0805_2012Metric, symbol LiBCM-rescue:R
Connections:
- net CELL18pos: now also R359.2; no longer J16.1 (Pin_1)
- net IP_ISO_STAR: no longer R223.1, R340.1, R341.1, R344.1, R347.1, R350.1, R353.1, R355.1
- net ISOA_TAP: no longer R175.1, T2.7
- new net CELL19neg: J16.1 (Pin_1), R359.1
- new net IM_ISO_STAR: R223.1, R340.1, R341.1, R344.1, R347.1, R350.1, R353.1, R355.1
- new net ISOB_TAP: R175.1, T2.7
Other:
- note added: "SNUBBER DOESN'T\nFIT. SHORT TRACES"
Changed lines of the file:
@@
 BIAS_B
 Text Label 10200 14700 1    60   ~ 0
-ISOA_TAP
+ISOB_TAP
 Wire Wire Line
 	15700 15750 15700 15500
@@
 	5300 4300 5250 4300
 Wire Wire Line
-	7050 950  7050 7250
+	7050 950  7050 6525
 Text Notes 10250 8700 0    110  ~ 0
 U11/U12/U13 ARE NOT\nGALVANICALLY ISOLATED
@@
 IP_ISO_SAFETY
 Text Label 7850 15750 2    60   ~ 0
-IP_ISO_STAR
+IM_ISO_STAR
 Text Label 8600 15200 0    60   ~ 0
 IP_TERMA
@@
 	18000 13650 18250 13650
 Wire Wire Line
-	24050 14600 24200 14600
-$Comp
-L LiBCM-rescue:C C176
-U 1 1 A38B0068
-P 24200 14400
-F 0 "C176" H 24225 14500 50  0000 L CNN
-F 1 "DNP" H 24225 14300 50  0000 L CNN
-F 2 "Capacitor_SMD:C_0805_2012Metric" H 24238 14250 50  0001 C CNN
-F 3 "" H 24200 14400 50  0000 C CNN
-	1    24200 14400
-	1    0    0    1
-$EndComp
-Wire Wire Line
-	24200 14600 24200 14550
-Connection ~ 24200 14600
-Wire Wire Line
-	24200 14600 24450 14600
-Wire Wire Line
-	24200 14250 24200 13950
-Text Label 24200 13950 3    60   ~ 0
-SNUBD
-Wire Wire Line
-	24050 13600 24200 13600
-$Comp
-L LiBCM-rescue:R R351
-U 1 1 A38B0076
-P 24200 13800
-F 0 "R351" V 24280 13800 50  0000 C CNN
-F 1 "DNP" V 24200 13800 50  0000 C CNN
-F 2 "Resistor_SMD:R_0805_2012Metric" V 24130 13800 50  0001 C CNN
-F 3 "" H 24200 13800 50  0000 C CNN
-	1    24200 13800
-	1    0    0    -1
-$EndComp
-Wire Wire Line
-	24200 13650 24200 13600
-Connection ~ 24200 13600
-Wire Wire Line
-	24200 13600 24450 13600
-Wire Wire Line
 	30250 14500 30400 14500
 $Comp
@@
 Wire Wire Line
 	1200 14850 1750 14850
+$Comp
+L LiBCM-rescue:R R359
+U 1 1 61A07E3A
+P 7050 6675
+F 0 "R359" V 7130 6675 50  0000 C CNN
+F 1 "20" V 7050 6675 50  0000 C CNN
+F 2 "Resistor_SMD:R_0805_2012Metric" V 6980 6675 50  0001 C CNN
+F 3 "" H 7050 6675 50  0000 C CNN
+	1    7050 6675
+	1    0    0    -1
+$EndComp
+Text Label 7050 6125 1    60   ~ 0
+CELL19neg
+Wire Wire Line
+	7050 6825 7050 7250
+Wire Wire Line
+	24050 13600 24450 13600
+Wire Wire Line
+	24050 14600 24450 14600
+Text Notes 24325 14550 1    59   ~ 0
+SNUBBER DOESN'T\nFIT.  SHORT TRACES
 $EndSCHEMATC
