File: Electronics/PCB (KiCAD)/RevC/KiCAD/LiBCM.kicad_pcb (KiCad board)
At the start: 4 copper layers, 355 x 160 mm, 624 parts, among them J1 Conn_01x08, J10 Screw_Terminal_01x03, J11 Screw_Terminal_01x08, J12 Conn_01x02_Male, J13 Conn_01x20, J14 Conn_01x04, J15 Conn_01x02, J16 Conn_01x20, J17 Conn_01x14, J18 Conn_01x14, J2 Conn_01x08, J3 Conn_01x08, J4 Conn_02x03_Odd_Even, J5 Conn_01x08, J6 Conn_01x08, J7 Conn_01x08, J8 Screw_Terminal_01x06, J9 Screw_Terminal_01x08, M1 Fan, M2 Fan, M3 Fan, P1 OEM_BCM_Connector, P2 Conn_WallPlug_Earth, Q1 Q_NMOS_GSD, Q10 Q_PMOS_GSD, Q11 Q_PMOS_GSD, Q12 Q_PMOS_GSD, Q13 Q_PMOS_GSD, Q14 Q_PMOS_GSD, Q15 Q_PMOS_GSD, Q16 Q_PMOS_GSD, Q17 Q_PMOS_GSD, Q18 Q_PMOS_GSD, Q19 Q_PMOS_GSD, Q2 Q_NMOS_GSD, Q20 Q_NPN_BCEC, Q21 Q_PMOS_GSD, Q22 Q_PMOS_GSD, Q23 Q_PMOS_GSD, Q24 Q_PMOS_GSD, Q25 Q_PMOS_GSD, Q26 Q_PMOS_GSD, Q27 Q_PMOS_GSD, Q28 Q_PMOS_GSD, Q29 Q_PMOS_GSD, Q3 Q_NMOS_GSD, Q30 Q_PMOS_GSD, Q31 Q_PMOS_GSD, Q32 Q_PMOS_GSD, Q33 Q_NPN_BCEC, Q34 Q_PMOS_GSD, Q35 Q_PMOS_GSD, Q36 Q_PMOS_GSD, Q37 Q_PMOS_GSD, Q38 Q_PMOS_GSD, Q39 Q_PMOS_GSD, Q4 Q_NMOS_GSD, Q40 Q_PMOS_GSD, Q41 Q_PMOS_GSD, Q42 Q_PMOS_GSD, Q43 Q_PMOS_GSD, Q44 Q_PMOS_GSD, Q45 Q_PMOS_GSD, Q46 Q_NPN_BCEC, Q47 Q_PMOS_GSD, Q48 Q_PMOS_GSD, Q49 Q_PMOS_GSD, Q5 Q_NMOS_GSD, Q50 Q_PMOS_GSD, Q51 Q_PMOS_GSD, Q52 Q_PMOS_GSD, Q53 Q_PMOS_GSD, Q54 Q_PMOS_GSD, Q55 Q_PMOS_GSD, Q56 Q_PMOS_GSD, Q57 Q_PMOS_GSD, Q58 Q_PMOS_GSD, Q59 Q_NPN_BCEC, Q6 Q_NMOS_GSD, Q60 Q_PMOS_GSD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

Commit message: RevC PCB in Layout
Parts:
- removed REF**: OSHW-Logo_11.4x12mm_SilkScreen, Symbol:OSHW-Logo_11.4x12mm_SilkScreen
- added BZ1: Buzzer, Linsight:BUZZER_WT-1205, F.Cu at (184.8, 84.8)
- added C157: 1u, Capacitor_SMD:C_0805_2012Metric, F.Cu at (215.2, 25.0)
- added C158: 1u, Capacitor_SMD:C_0805_2012Metric, F.Cu at (18.8, 106.2)
- added C159: 100p, Capacitor_SMD:C_0805_2012Metric, F.Cu at (101.0, 146.2)
- added C160: 100p, Capacitor_SMD:C_0805_2012Metric, F.Cu at (101.8, 140.5)
- added C161: 100p, Capacitor_SMD:C_0805_2012Metric, F.Cu at (135.6, 100.0)
- added C162: 100p, Capacitor_SMD:C_0805_2012Metric, F.Cu at (140.5, 96.0)
- added C163: 100p, Capacitor_SMD:C_0805_2012Metric, F.Cu at (156.3, 136.0)
- added C164: 1u, Capacitor_SMD:C_0805_2012Metric, F.Cu at (143.8, 108.0)
- added C165: 100n, Capacitor_SMD:C_0805_2012Metric, F.Cu at (315.2, 62.5)
- added C166: 1u, Capacitor_SMD:C_0805_2012Metric, F.Cu at (143.9, 111.6)
- added C167: 1u, Capacitor_SMD:C_0805_2012Metric, F.Cu at (143.9, 115.0)
- added C168: 1u, Capacitor_SMD:C_0805_2012Metric, F.Cu at (143.9, 118.4)
- added C169: 100n, Capacitor_SMD:C_0805_2012Metric, F.Cu at (142.8, 138.9)
- added C170: 100n, Capacitor_SMD:C_0805_2012Metric, F.Cu at (145.8, 87.2)
- added C171: 100n, Capacitor_SMD:C_0805_2012Metric, F.Cu at (157.5, 97.5)
- added C172: 100p, Capacitor_SMD:C_0805_2012Metric, F.Cu at (151.5, 98.5)
- added C173: DNP, Capacitor_SMD:C_0805_2012Metric, F.Cu at (30.2, 74.5)
- added C174: DNP, Capacitor_SMD:C_0805_2012Metric, F.Cu at (64.5, 171.0)
- added C175: DNP, Capacitor_SMD:C_0805_2012Metric, F.Cu at (174.0, 180.2)
- added C177: DNP, Capacitor_SMD:C_0805_2012Metric, F.Cu at (283.5, 171.0)
- added D18: D, Diode_SMD:D_SMA, F.Cu at (369.5, 40.0)
- added J19: Conn_02x02, Linsight:CONN_WM26831CT-ND​, F.Cu at (211.0, 26.2)
- added J20: Conn_02x02, Linsight:CONN_WM26831CT-ND​, F.Cu at (306.5, 20.5)
- added J21: Conn_01x04, Connector_PinHeader_2.54mm:PinHeader_1x04_P2.54mm_Vertical, F.Cu at (159.0, 152.8)
- added J22: Conn_01x08, Connector_PinSocket_2.54mm:PinSocket_1x08_P2.54mm_Vertical, F.Cu at (142.2, 153.2)
- added Q73: Q_NMOS_GSD, Package_TO_SOT_SMD:SOT-23, F.Cu at (169.5, 91.0)
- added Q77: Q_PMOS_GSD, Package_TO_SOT_SMD:SOT-23, F.Cu at (142.8, 136.0)
- added R12: 1k24, Resistor_SMD:R_0805_2012Metric, F.Cu at (190.2, 23.8)
- added R14: 1k24, Resistor_SMD:R_0805_2012Metric, F.Cu at (282.0, 19.5)
- added R15: 7k32, Resistor_SMD:R_0805_2012Metric, F.Cu at (167.5, 94.0)
- added R318: 7k32, Resistor_SMD:R_0805_2012Metric, F.Cu at (137.9, 102.4)
- added R321: 100, Resistor_SMD:R_0805_2012Metric, F.Cu at (141.2, 99.0)
- added R322: 100, Resistor_SMD:R_0805_2012Metric, F.Cu at (141.8, 102.4)
- added R323: 71k5, Resistor_SMD:R_0805_2012Metric, F.Cu at (116.0, 115.5)
- added R324: 71k5, Resistor_SMD:R_0805_2012Metric, F.Cu at (129.5, 141.2)
- added R325: 100, Resistor_SMD:R_0805_2012Metric, F.Cu at (156.3, 139.4)
- added R326: 1k24, Resistor_SMD:R_0805_2012Metric, F.Cu at (156.3, 132.6)
- added R327: 20, Resistor_SMD:R_0805_2012Metric, F.Cu at (317.2, 59.5)
- added R328: DNP, Resistor_SMD:R_0805_2012Metric, F.Cu at (132.2, 123.5)
- added R329: DNP, Resistor_SMD:R_0805_2012Metric, F.Cu at (132.2, 132.0)
- added R330: 100, Resistor_SMD:R_0805_2012Metric, F.Cu at (336.8, 68.5)
- added R331: 100, Resistor_SMD:R_0805_2012Metric, F.Cu at (254.8, 42.5)
- added R332: 100, Resistor_SMD:R_0805_2012Metric, F.Cu at (320.8, 52.5)
- added R333: 100, Resistor_SMD:R_0805_2012Metric, F.Cu at (336.8, 73.0)
- added R334: 100, Resistor_SMD:R_0805_2012Metric, F.Cu at (155.0, 97.5)
- added R335: 10k, Resistor_SMD:R_0805_2012Metric, F.Cu at (341.2, 58.0)
- added R336: 10k, Resistor_SMD:R_0805_2012Metric, F.Cu at (348.8, 60.5)
- added R337: 100, Resistor_SMD:R_0805_2012Metric, F.Cu at (271.5, 42.2)
- added R338: DNP, Resistor_SMD:R_0805_2012Metric, F.Cu at (30.2, 77.0)
- added R339: 20, Resistor_SMD:R_0805_2012Metric, F.Cu at (354.2, 185.5)
- added R340: 20, Resistor_SMD:R_0805_2012Metric, F.Cu at (356.8, 185.5)
- added R341: 20, Resistor_SMD:R_0805_2012Metric, F.Cu at (49.5, 189.2)
- added R342: 20, Resistor_SMD:R_0805_2012Metric, F.Cu at (47.0, 189.2)
- added R343: 20, Resistor_SMD:R_0805_2012Metric, F.Cu at (68.2, 189.5)
- added R344: 20, Resistor_SMD:R_0805_2012Metric, F.Cu at (70.8, 189.5)
- added R345: DNP, Resistor_SMD:R_0805_2012Metric, F.Cu at (60.5, 171.0)
- added R346: 20, Resistor_SMD:R_0805_2012Metric, F.Cu at (266.8, 189.5)
- added R347: 20, Resistor_SMD:R_0805_2012Metric, F.Cu at (269.2, 189.5)
- added R348: DNP, Resistor_SMD:R_0805_2012Metric, F.Cu at (171.5, 180.3)
- added R349: 20, Resistor_SMD:R_0805_2012Metric, F.Cu at (344.0, 188.5)
- added R350: 20, Resistor_SMD:R_0805_2012Metric, F.Cu at (352.2, 188.8)
- added R352: 20, Resistor_SMD:R_0805_2012Metric, F.Cu at (288.8, 189.5)
- added R353: 20, Resistor_SMD:R_0805_2012Metric, F.Cu at (291.2, 189.5)
- added R354: 100, Resistor_SMD:R_0805_2012Metric, F.Cu at (42.1, 186.4)
- added R355: 100, Resistor_SMD:R_0805_2012Metric, F.Cu at (44.5, 186.4)
- added R356: 20, Resistor_SMD:R_0805_2012Metric, F.Cu at (43.1, 183.2)
- added R357: DNP, Resistor_SMD:R_0805_2012Metric, F.Cu at (280.8, 171.0)
- added R358: DNP, Resistor_SMD:R_0805_2012Metric, F.Cu at (139.3, 136.2)
- added R359: 20, Resistor_SMD:R_0805_2012Metric, F.Cu at (118.2, 161.8)
- added R4: 1k24, Resistor_SMD:R_0805_2012Metric, F.Cu at (-13.2, 106.0)
- C101, C102, C155: value 22n -> 1u; footprint Capacitor_SMD:C_1206_3216Metric -> Capacitor_SMD:C_0805_2012Metric
- C103, C142, C48, C52, C77, C93: value 20p -> 100p
- C104, C105, C106, C107, C108, C109, C110, C111, C112, C113, C114, C115, C116, C122, C123, C124, C125, C126, C127, C128, C129, C130, C131, C132, C133, C134, C3, C35, C36, C37, C38, C39, C40, C41, C42, C43, C44, C45, C46, C47, C57, C58, C59, C60, C61, C62, C63, C64, C65, C66, C67, C68, C69, C79, C80, C81, C82, C83, C84, C85, C86, C87, C88, C89, C90, C91: value 10n -> 100n
- C12, C5, C6, C7, C9: value 100n -> 1u
- C151: value 22n -> 68n
- C152: value 68n -> 22n
- C156: value DNP -> 1u
- D16: value LED -> 1N4148W; footprint LED_SMD:LED_0805_2012Metric_Castellated -> Diode_SMD:D_SOD-123
- J10: value Screw_Terminal_01x03 -> Screw_Terminal_01x01; footprint Connector_Wire:SolderWire-1sqmm_1x03_P5.4mm_D1.4mm_OD2.7mm -> Connector_Wire:SolderWire-1sqmm_1x01_D1.4mm_OD2.7mm
- J12: value Conn_01x02_Male -> Conn_02x02; footprint Connector_Wire:SolderWire-0.25sqmm_1x02_P4.2mm_D0.65mm_OD1.7mm -> Linsight:CONN_WM26831CT-ND​
- J14: footprint Connector_PinHeader_2.54mm:PinHeader_1x04_P2.54mm_Vertical -> Connector_PinSocket_2.54mm:PinSocket_1x04_P2.54mm_Horizontal
- J4: value Conn_02x03_Odd_Even -> Conn_02x08_Odd_Even; footprint Connector_PinHeader_2.54mm:PinHeader_2x03_P2.54mm_Vertical -> Connector_PinHeader_2.54mm:PinHeader_2x08_P2.54mm_Vertical; moved to F.Cu
- J8: value Screw_Terminal_01x06 -> Conn_01x04; footprint Connector_PinHeader_2.54mm:PinHeader_1x06_P2.54mm_Vertical -> Connector_PinHeader_2.54mm:PinHeader_1x04_P2.54mm_Vertical
- R1, R122, R2, R3, R43, R44, R45, R46, R5: value 1k -> 1k24
- R10, R11, R7, R8, R9: value 3k3 -> DNP
- R100, R101, R102, R103, R104, R105, R106, R107, R123, R124, R144, R145, R146, R147, R148, R149, R150, R151, R152, R153, R154, R155, R156, R16, R169, R170, R189, R190, R191, R192, R193, R194, R195, R196, R197, R198, R199, R200, R201, R216, R217, R23, R237, R238, R239, R240, R241, R242, R243, R244, R245, R246, R247, R248, R249, R262, R263, R278, R279, R280, R281, R282, R283, R284, R285, R286, R287, R288, R289, R290, R303, R304, R50, R95, R96, R97, R98, R99: value 82 -> 100
- R108, R109, R110, R111, R112, R113, R114, R115, R116, R117, R118, R119, R157, R158, R159, R160, R161, R162, R163, R164, R165, R166, R167, R168, R202, R203, R204, R205, R206, R207, R208, R209, R210, R211, R212, R213, R250, R251, R252, R253, R254, R255, R256, R257, R258, R259, R260, R261, R291, R292, R293, R294, R295, R296, R297, R298, R299, R300, R301, R302: value 3.3k -> 1k24
- R120, R126, R172, R219, R265, R306: value 1k -> 768
- R121: value 120 -> 1k24
- R125, R171, R218, R264, R305: value 3k3 -> 7k32
- R128, R174, R221, R24, R25, R267, R28, R308, R31, R320, R60, R81: value 3k3 -> 1k24
- R130: value 100k -> 5M
- R17, R223, R311, R68: value 120 -> 100
- R19, R48: value DNP -> 10k
- R26, R319, R39, R42, R47: value 10k -> 7k32
- R29: value 120 -> 768
- R30: value 120 -> 20
- R313: value DNP -> 100
- R314: value DNP -> 20
- R316, R53: value 82 -> 768
- R317: value 82 -> 7k32
- R33: value 3k3 -> 768
- R40, R41: value 120 -> DNP
- R54, R59, R63, R65, R78: value 220 -> 100
- R58: value 1k -> 10k
- R69, R72: value 10k@0.25W -> 10k
- R70, R71: value 20k@0.5W -> 10k
- R80: value DNP -> 71k5
- R82: value 100k -> 100
- SW1: footprint Button_Switch_SMD:Panasonic_EVQPUJ_EVQPUA -> Button_Switch_Keyboard:SW_Cherry_MX_1.00u_PCB
- moved C155 378.4 mm to (-9.20, 106.0), turned to 90 degrees
- moved C101 292.7 mm to (286.0, 19.5), turned to 90 degrees
- moved R314 260.3 mm to (101.8, 143.0), turned to 180 degrees
- moved C102 211.7 mm to (193.0, 24.0), turned to 90 degrees
- moved R80 195.9 mm to (161.8, 151.0), turned to 270 degrees
- moved R19 188.8 mm to (297.8, 19.8), turned to 270 degrees
- moved C156 168.8 mm to (311.5, 20.0), turned to 90 degrees
- moved R313 166.2 mm to (105.8, 143.0), turned to 0 degrees
- moved D16 165.4 mm to (172.8, 89.8)
- moved R58 151.9 mm to (4.80, 105.5), turned to 270 degrees
- moved R49 134.6 mm to (277.0, 74.5), turned to 270 degrees
- moved R48 115.5 mm to (202.8, 25.2), turned to 270 degrees
- moved R13 112.3 mm to (133.8, 44.5), turned to 180 degrees
- moved Q1 110.4 mm to (133.8, 47.8), turned to 270 degrees
- moved C2 108.9 mm to (149.2, 52.2), turned to 0 degrees
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Connections:
- net /12NEG_UNFILTERED renamed /12NEG_RAW
- net /12POS_UNFILTERED renamed /12POS_RAW
- net /HLINE_JUMPER renamed /HLINE
- net /LOAD5V_R renamed /5VP_GATE
- net /LiBCM BMS/IM_ISO_A renamed /LiBCM BMS/IM_ISOA_X
- net /LiBCM BMS/IM_ISO_B renamed /LiBCM BMS/IM_ISOB_X
- net /LiBCM BMS/IM_ISO_C renamed /LiBCM BMS/IM_ISOC_X
- net /LiBCM BMS/IM_ISO_D renamed /LiBCM BMS/IM_ISOD_X
- net /LiBCM BMS/IM_ISO_E renamed /LiBCM BMS/IM_ISOE_X
- net /LiBCM BMS/IP_ISO_A renamed /LiBCM BMS/IP_ISOA_X
- net /LiBCM BMS/IP_ISO_B renamed /LiBCM BMS/IP_ISOB_X
- net /LiBCM BMS/IP_ISO_C renamed /LiBCM BMS/IP_ISOC_X
- net /LiBCM BMS/IP_ISO_D renamed /LiBCM BMS/IP_ISOD_X
- net /LiBCM BMS/IP_ISO_E renamed /LiBCM BMS/IP_ISOE_X
- net /LiBCM BMS/ISO_TAP_A renamed /LiBCM BMS/ISOA_TAP
- net /LiBCM BMS/ISO_TAP_B renamed /LiBCM BMS/ISOB_TAP
- net /LiBCM BMS/ISO_TAP_C renamed /LiBCM BMS/ISOC_TAP
- net /LiBCM BMS/ISO_TAP_D renamed /LiBCM BMS/ISOD_TAP
- net /LiBCM BMS/ISO_TAP_E renamed /LiBCM BMS/ISOE_TAP
- net /TBATT_BLU renamed /TEMP_BLU
- net /TBATT_BLU_LPF renamed /TEMP_BLU_LPF
- net /TBATT_GRN renamed /TEMP_GRN
- net /TBATT_GRN_LPF renamed /TEMP_GRN_LPF
- net /TBATT_WHT renamed /TEMP_WHT
- net /TBATT_WHT_LPF renamed /TEMP_WHT_LPF
- net /TBATT_YEL renamed /TEMP_YEL
- net /TBATT_YEL_LPF renamed /TEMP_YEL_LPF
- C101 pad 1: /LiBCM BMS/IP_ISO_SAFETY -> GND_ENG
- C101 pad 2: /LiBCM BMS/IP_ISO_EXT -> /TBATT_BAY1_LPF
- C102 pad 1: /LiBCM BMS/IM_ISO_SAFETY -> GND_ENG
- C102 pad 2: /LiBCM BMS/IM_ISO_EXT -> /TBATT_BAY2_LPF
- C140 pad 1: /LiBCM BMS/IP_ISO_SAFETY -> /LiBCM BMS/IP_TERME
- C141 pad 1: /LiBCM BMS/IM_ISO_SAFETY -> /LiBCM BMS/IM_TERME
- C15 pad 1: +5V -> GND_ENG
- C15 pad 2: GND_ENG -> +5V
- C155 pad 2: /LiBCM BMS/TCENTER_ISO_SAFETY -> /TBATT_BAY3_LPF
- C156 pad 1: /FAN_PWM_G -> GND_ENG
- C156 pad 2: GND_ENG -> /TBATT_BAY1
- C16 pad 1: +5V -> GND_ENG
- C16 pad 2: GND_ENG -> +5V
- C48 pad 1: GND_ENG -> /LiBCM BMS/TCENTER_6820
- C48 pad 2: /LiBCM BMS/TCENTER_6820 -> GND_ENG
- C55 pad 1: /LiBCM BMS/IM_ISO_SAFETY -> /LiBCM BMS/IM_TERMA
- C56 pad 1: /LiBCM BMS/IP_ISO_SAFETY -> /LiBCM BMS/IP_TERMA
- C71 pad 1: /LiBCM BMS/IP_ISO_SAFETY -> /LiBCM BMS/IP_TERMB
- C72 pad 1: /LiBCM BMS/IM_ISO_SAFETY -> /LiBCM BMS/IM_TERMB
- C78 pad 1: /LiBCM BMS/IP_ISO_SAFETY -> /LiBCM BMS/IP_TERMC
- C92 pad 1: /LiBCM BMS/IM_ISO_SAFETY -> /LiBCM BMS/IM_TERMC
- C95 pad 1: /LiBCM BMS/IP_ISO_SAFETY -> /LiBCM BMS/IP_TERMD
- C96 pad 1: /LiBCM BMS/IM_ISO_SAFETY -> /LiBCM BMS/IM_TERMD
- D16 pad 1: /MCM_E_LED_A -> +5V
- D16 pad 2: /MCM_E_CONTROL -> /BUZ1
- D6 pad 2: /L1_FUSED -> /L1
- F1 pad 1: /L1_FUSED -> /L1
- F1 pad 2: /L1 -> /L1_UNFUSED
- H2 pad 1: GND_ENG -> Net-(H2-Pad1)
- H7 pad 1: GND_ENG -> Net-(H7-Pad1)
- J11 pad 4: HVDC_POS_FUSED -> /GRID_HVDC+
- J12 pad 1: /LiBCM BMS/IM_ISO_EXT -> /TBATT_BAY3
- J12 pad 2: /LiBCM BMS/IP_ISO_EXT -> /TEMP_NEG
- J16 pad 1: /LiBCM BMS/CELL18pos -> /LiBCM BMS/CELL19neg
- J2 pad 1: /BATT_CURRENT_SCALED -> /BATT_CURRENT_ADC
- J3 pad 2: /HMI_EN -> /TBATT_BAY1_LPF
- J3 pad 3: /BATTSCI_DE -> /TBATT_BAY2_LPF
- J3 pad 4: /BATTSCI_REn -> /TBATT_BAY3_LPF
- J3 pad 7: /LED3 -> /GPIO-1
- J3 pad 8: /LED4 -> /GPIO-2
- J4 pad 1: /GPIO-1 -> /BATTSCI_DE
- J4 pad 2: /USER_SW -> /BATTSCI_REn
- J4 pad 3: /SPI_BATT_MISO -> /GPIO-0
- J4 pad 4: /SPI_BATT_MOSI -> /COVER_SWITCH
- J4 pad 5: /SPI_BATT_SCK -> /BUZZER
- J4 pad 6: /SPI_BATT_CS0 -> /GPIO-3
- J5 pad 5: /I_SENSOR_EN -> /HMI_EN
- J6 pad 5: /VPIN_OUT_PWM -> /USER_SW
- J6 pad 6: /SPI_EXTERNAL_CS1 -> /VPIN_OUT_PWM
- J6 pad 7: /TEMP_SENSOR_EN -> /SENSOR_EN
- J8 pad 1: /SDA -> +5V
- J8 pad 2: /SCL -> /SCLc
- J8 pad 3: +5V -> /SDAc
- J8 pad 4: /GPIO-1 -> GND_ENG
- P1 pad A01: /IGNITION_12V -> /12V_KEYON
- P1 pad A02: /IGNITION_12V -> /12V_KEYON
- P1 pad B02: /SPI_BATT_MISO -> Net-(P1-PadB02)
- P1 pad B03: /SPI_BATT_MOSI -> Net-(P1-PadB03)
- P1 pad B04: /SPI_BATT_SCK -> Net-(P1-PadB04)
- P1 pad B05: /SPI_EXTERNAL_CS1 -> Net-(P1-PadB05)
- P1 pad B12: /TBATT_SG -> /TEMP_NEG
- P2 pad 1: /L1 -> /L1_UNFUSED
- Q3 pad 1: /I_SENSOR_EN -> /SENSOR_EN
- Q4 pad 1: /TEMP_SENSOR_EN -> /TEMP_EN
- Q4 pad 3: /TBATT_SG -> /TEMP_NEG
- Q7 pad 1: /FAN_PWM_G -> /FAN_PWM
- Q74 pad 1: /I_SENSOR_EN -> /SENSOR_EN
- Q76 pad 1: /I_SENSOR_EN -> /SENSOR_EN
- R121 pad 1: /LiBCM BMS/IP_6820 -> /SDA
- R121 pad 2: /LiBCM BMS/IM_6820 -> +5V
- R130 pad 1: /LiBCM BMS/TCENTER_ISO_SAFETY -> GND_ENG
- R130 pad 2: GND_ENG -> /LiBCM BMS/TCENTER_ISO_SAFETY
- R19 pad 1: /I_SENSOR_EN -> +5V
- R19 pad 2: /IGNITION_SENSE -> /TBATT_BAY1
- R21 pad 1: /IGNITION_DIV -> /KEYON_DIV
- R223 pad 1: /LiBCM BMS/IM_ISO_SAFETY -> /LiBCM BMS/IM_ISO_STAR
- R223 pad 2: /LiBCM BMS/IP_ISO_SAFETY -> /LiBCM BMS/IP_ISO_STAR
- R26 pad 1: /I_SENSOR_EN -> /SENSOR_EN
- R313 pad 1: +12V -> /SDAd
- R313 pad 2: /IGNITION_12V -> /SDA
- R314 pad 1: /MCM_E_E -> /SDAd
- R314 pad 2: /MCM_E_C -> /SDAc
- R316 pad 2: /SENSE_MID -> /I_SENSOR_RAW
- R317 pad 2: /SENSE_MID -> /SPI_MOSI
- R32 pad 2: /IGNITION_12V -> /12V_KEYON
- R39 pad 1: /TEMP_SENSOR_EN -> /TEMP_EN
- R40 pad 2: /METSCI1 -> /MET_T
- R41 pad 2: /BATTSCI1 -> /BAT_T
- R43 pad 1: +5V -> +5VP
- R45 pad 1: +5V -> +5VP
- R48 pad 1: /VPIN_IN_NOISY -> +5V
- R48 pad 2: /VPIN_OUT_LPF -> /TBATT_BAY2
- R49 pad 1: /FAN_PWM_G -> /FAN_PWM
- R50 pad 1: /SENSE_MID -> +5V
- R53 pad 1: /SENSE_MID -> +5V
- R58 pad 1: /FAN_PWM -> +5V
- R58 pad 2: /FAN_PWM_G -> /TBATT_BAY3
- R59 pad 2: /GRID_EN_LED_C -> /GRID_EN_DIV
- R6 pad 1: /IGNITION_12V -> /KEYON_DIV
- R6 pad 2: /IGNITION_DIV -> /12V_KEYON
- R63 pad 1: GND_ENG -> /GRID_PWM_DIV
- R63 pad 2: /GRID_PWM_LED_C -> GND_ENG
- R67 pad 1: /BATT_CURRENT_SCALED -> /OP_OUT
- R70 pad 2: /MCM_E_CONN+ -> /MCM_E_C2
- R71 pad 1: /MCM_E_CONN- -> /MCM_E_E2
- R73 pad 1: /L1_FUSED -> /L1
- R74 pad 1: /L1_FUSED -> /L1
- R75 pad 1: /L1_FUSED -> /L1
- R76 pad 2: /L1_FUSED -> /L1
- R78 pad 1: /L1_GRID -> /L1_SNUB
- R80 pad 1: /GRID_PWM+ -> /COVER_SWITCH
- R80 pad 2: /GRID_PWM- -> GND_ENG
- R81 pad 1: +5V -> /SCL
- R81 pad 2: /SPI_BATT_MISO -> +5V
- R82 pad 1: +5V -> /SCLc
- R82 pad 2: /SPI_BATT_MOSI -> /SCL
- SW1 pad 1: /FAN_PWM_G -> /COVER_SWITCH
- U10 pad 2: /SPI_BATT_MOSI -> /SPI_MOSI_FILT
- U10 pad 3: /SPI_BATT_MISO -> /SPI_MISO_FILT
- U10 pad 4: /SPI_BATT_SCK -> /SPI_SCK_FILT
- U10 pad 5: /SPI_BATT_CS0 -> /SPI_CS_LTC
- U4 pad 1: /BATT_CURRENT_SCALED -> /OP_OUT
Routing:
- net GND_ENG: track 3555.4 -> 2776.1 mm, vias 697 -> 548
- net /LiBCM BMS/IP_ISO_SAFETY: track 420.8 -> 2.97 mm, vias 6 -> 0
- net /LiBCM BMS/IM_ISO_SAFETY: track 419.6 -> 4.03 mm, vias 5 -> 0
- net /LiBCM BMS/IP_ISO_STAR: track 0.00 -> 342.4 mm, vias 0 -> 7
- net /LiBCM BMS/IM_ISO_STAR: track 0.00 -> 335.4 mm, vias 0 -> 7
- net /I_SENSOR_EN: track 245.9 -> 0.00 mm, vias 4 -> 0
- net /FAN_PWM_G: track 193.4 -> 0.00 mm, vias 2 -> 0
- net /SPI_BATT_MISO: track 179.1 -> 0.00 mm, vias 1 -> 0
- net /SPI_BATT_MOSI: track 176.5 -> 0.00 mm, vias 1 -> 0
- net /SPI_BATT_SCK: track 163.0 -> 0.00 mm, vias 1 -> 0
- net /IGNITION_12V: track 157.5 -> 0.00 mm, vias 2 -> 0
- net /SENSOR_EN: track 0.00 -> 151.6 mm
- net /HLINE_CONN: track 224.0 -> 86.8 mm, vias 6 -> 2
- net /TEMP_SENSOR_EN: track 131.0 -> 0.00 mm, vias 2 -> 0
- net +5V: track 723.5 -> 594.5 mm, vias 26 -> 13
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- added copper zone on F.Cu, net /L1
- removed copper zone on F.Cu, net /FAN_PWM_G
- removed copper zone on F.Cu, net /L1_FUSED
Other:
- board text added: "18S BAY3"
- board text added: "4A@300VAC"
- board text added: "4A@300VDC"
- board text added: "BAY3 MODULES"
- board text added: "DANGER:"
- board text added: "DANGER: HVDC WHEN IMA SWITCH ON OR GRID CHARGER POWERED"
- board text added: "DIM+ DIM- GRID- GRID+ MCMe+ MCMe- PACK- PA"
- board text added: "FAILURE TO FOLLOW THESE RULES WILL DESTROY IC U12: DO NOT PLACE FUSE/SWITCH BETWEEN CELLS C1:C36!!!!! CONNECT HIGH CURRENT CABLES TO CELLS C1:C36 BEFORE J13/J16 DISCONNECT J13/J16 BEFORE C1:C36 HIGH CURRENT CABLES"
- board text added: "GND GND CS IO-0 MISO CLK MOSI 5V"
- board text added: "GND SDA SCL 5V"
- board text added: "HAZARDOUS"
- board text added: "HVDC DANGER"
- board text added: "IMA SWITCH IS OFF"
- board text added: "L(GRID)"
- board text added: "LOCK USER"
- board text added: "NC IOREF RESET 3V3 5V0 GND GND VIN"
- board text added: "OD TX RX 5V"
- board text added: "PLUGGED IN"
- board text added: "PRESENT EVEN WHEN"
- board text added: "RevC"
- board text added: "VOLTAGE PRESENT WHEN BAY2 OR"
- board text removed: "*SWITCHED GROUND"
- board text removed: "12S/18S BAY3"
- board text removed: "C61-72: 0x7 C73-84: 0x8"
- board text removed: "DANGER!!"
- board text removed: "DANGER: HAZARDOUS VOLTAGE PRESENT EVEN WHEN IMA SWITCH IS OFF"
- board text removed: "DEBUG"
- board text removed: "FAILURE TO FOLLOW THESE RULES WILL DESTROY IC U12: DO NOT PLACE FUSE/SWITCH BETWEEN CELLS C1:C36!!!!! CONNECT CELLS C1:C36 TOGETHER WITH HIGH CURRENT CABLES BEFORE CONNECTING J13/J16 DISCONNECT J13/J16 BEFORE REMOVING HIGH CURRENT CABLES BETWEEN C1:C36"
- board text removed: "GND N L(GRID)"
- board text removed: "GRIDPWM+ GRIDPWM- GRID_DC- GRID_DC+ MCM_E+ MCM_E- PACK- PA"
- board text removed: "HAZARDOUS VOLTAGE PRESENT EVEN"
- board text removed: "HVDC WHEN LT DC1942C CONNECTED"
- board text removed: "NC IOREF RESET 3V3 5V0 GNDENG GNDENG VIN"
- board text removed: "OD* TX RX 5V"
- board text removed: "P M"
- board text removed: "PROGRAM OPTION"
- board text removed: "RevB"
- board text removed: "SDA SCL 5V IO1 GND GND"
- board text removed: "WHEN IMA SWITCH IS OFF"
- board text removed: "isoSPI"

Commit message: RevC PCB
Parts:
- added REF**: OSHW-Logo_11.4x12mm_SilkScreen, Symbol:OSHW-Logo_11.4x12mm_SilkScreen, F.Cu at (37.2, 174.2)
- J12, J19, J20: moved to B.Cu
- moved C156 192.6 mm to (151.2, 126.8)
- moved R19 183.4 mm to (148.8, 126.8), turned to 90 degrees
- moved R4 169.4 mm to (153.8, 134.8), turned to 270 degrees
- moved C101 168.3 mm to (156.2, 126.8)
- moved C155 167.9 mm to (156.2, 134.8), turned to 270 degrees
- moved R14 167.2 mm to (153.8, 126.8)
- moved R58 146.9 mm to (148.8, 134.8)
- moved C158 135.5 mm to (151.2, 134.8), turned to 270 degrees
- moved C157 123.6 mm to (151.2, 130.8)
- moved R48 118.5 mm to (148.8, 130.8), turned to 90 degrees
- moved J12 118.0 mm to (128.0, 79.8), turned to 180 degrees
- moved R12 113.1 mm to (153.8, 130.8)
- moved C102 112.9 mm to (156.2, 130.8)
- moved R42 101.8 mm to (131.5, 118.8)
- moved R47 82.3 mm to (157.0, 118.5), turned to 90 degrees
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Connections:
- J2 pad 2: /BATTFANL_EN -> /USER_SW
- J2 pad 3: /BATTFANH_EN -> /VPIN_IN
- J2 pad 8: /VPIN_IN -> /BATTFANL_EN
- J3 pad 1: /TURN_OFF_5V -> /BATTFANH_EN
- J6 pad 5: /USER_SW -> /TURN_OFF_5V
Routing:
- net GND_ENG: track 2776.1 -> 3343.4 mm, vias 548 -> 594
- net /TEMP_NEG: track 99.3 -> 352.2 mm, vias 0 -> 8
- net +5V: track 594.5 -> 805.5 mm, vias 13 -> 24
- net /TBATT_BAY1: track 0.00 -> 192.0 mm, vias 0 -> 5
- net /LED1: track 0.11 -> 159.2 mm, vias 0 -> 2
- net /LED2: track 0.17 -> 157.3 mm, vias 0 -> 2
- net /LED3: track 2.12 -> 140.3 mm, vias 0 -> 2
- net /LED4: track 2.42 -> 140.3 mm, vias 0 -> 2
- net /TBATT_BAY2: track 0.00 -> 117.0 mm, vias 0 -> 5
- net /SENSOR_EN: track 151.6 -> 246.8 mm, vias 0 -> 1
- net /USER_SW: track 0.23 -> 81.6 mm, vias 0 -> 2
- net /TBATT_BAY3: track 0.00 -> 73.0 mm, vias 0 -> 3
- net /SPI_MISO_FILT: track 0.00 -> 60.3 mm, vias 0 -> 3
- net /SPI_MOSI: track 20.6 -> 71.8 mm, vias 0 -> 1
- net /SPI_CS_LTC: track 5.95 -> 56.4 mm, vias 0 -> 1
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- added copper zone on F.Cu, net /MCM_E_CONN+
- removed copper zone on B.Cu, net (none)
Other:
- board text added: "A TRULY GREAT TOOL LENDS ITSELF TO USES YOU NEVER EXPECTED"
- board text added: "DANGER"
- board text added: "DESIGNED BY 'MUDDER' FOR G1 HONDA INSIGHT GITHUB.COM/DOPPELHUB/HONDA_INSIGHT_LIBCM"
- board text added: "DISABLE RESET USER SWITCH"
- board text added: "FREE ROSS"
- board text added: "GND IO3 IO2 IO1"
- board text added: "NC IOREF RESET 3V3 5V0 GND VIN"
- board text added: "THE DOER ALONE LEARNS"
- board text added: "TO USE HLINE: -J14: SHORT TX & RX -J15: SHORT PINS -P1: CONNECT HLINE TO BCM CONN B01 TO USE LiDisplay: -J14: CONNECT CABLE -J15: REMOVE JUMPER"
- board text added: "WHAT I CANNOT CREATE I DO NOT UNDERSTAND"
- board text removed: "ARDUINO MEGA"
- board text removed: "DESIGNED BY 'MUDDER' FOR G1 HONDA INSIGHT INSIGHTCENTRAL.NET"
- board text removed: "GND_ENG"
- board text removed: "LOCK USER"
- board text removed: "NC IOREF RESET 3V3 5V0 GND GND VIN"
- board text removed: "TO USE LiDisplay: -J14: CONNECT CABLE -J15: REMOVE JUMPER TO USE HLINE: -J14: SHORT TX & RX -J15: SHORT PINS -P1: CONNECT HLINE TO BCM CONN B01"
