File: Electronics/PCB (KiCAD)/RevC/KiCAD/LiBCM.kicad_pcb (KiCad board)
At the start: 4 copper layers, 355 x 160 mm, 695 parts, among them J1 Conn_01x08, J10 Screw_Terminal_01x01, J11 Screw_Terminal_01x08, J12 Conn_02x02, J13 Conn_01x20, J14 Conn_01x04, J15 Conn_01x02, J16 Conn_01x20, J17 Conn_01x14, J18 Conn_01x14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

Commit message: Thinner Safety Cover
Also updated Fan cap to 2 uF, and generated centroids.
Parts:
- C145: value 22u -> 2u
