File: Electronics/PCB (KiCAD)/RevD/KiCAD/LiBCM.sch (KiCad schematic (older format))
At the start: 260 parts, among them J1 Conn_01x08, J10 Screw_Terminal_01x01, J11 Screw_Terminal_01x08, J12 Conn_02x02, J14 Conn_01x04, J15 Conn_01x02, J19 Conn_02x02, J2 Conn_01x08, J20 Conn_02x02, J21 Conn_01x04, J22 Conn_01x08, J3 Conn_01x08, J4 Conn_02x08_Odd_Even, J5 Conn_01x08, J6 Conn_01x08, J7 Conn_01x08, J8 Conn_01x04, J9 Screw_Terminal_01x08, M1 Fan, M2 Fan, M3 Fan, P1 OEM_BCM_Connector, P2 Conn_WallPlug_Earth, Q1 Q_NMOS_GSD, Q2 Q_NMOS_GSD, Q3 Q_NMOS_GSD, Q4 Q_NMOS_GSD, Q5 Q_NMOS_GSD, Q6 Q_NMOS_GSD, Q7 Q_NMOS_GSD, Q73 Q_NMOS_GSD, Q74 Q_NMOS_GSD, Q75 Q_PMOS_GSD, Q76 Q_NMOS_GSD, Q77 Q_PMOS_GSD, Q78 Q_NMOS_GSD, Q79 Q_NMOS_GSD, Q80 Q_NMOS_GSD, SW1 SW_Push, SW2 SW_DIP_x02, U1 AP63205WU, U16 AP62301, U2 LT1487, U3 LT1487, U4 LT1797, U5 MOC3023M, U6 SFH620A-2X007T, U7 SFH620A-2X007T, U8 EPM1510SJ, U9 H11D1SR2VM

Commit message: Finished RevD PCB (except for possible HVAC switch change)
Parts:
- removed J4: Conn_02x08_Odd_Even, Connector_PinHeader_2.54mm:PinHeader_2x08_P2.54mm_Vertical, symbol Connector_Generic:Conn_02x08_Odd_Even
- added C153: 22u, Capacitor_SMD:C_1210_3225Metric, symbol LiBCM-rescue:C
- added J4: Conn_02x09_Odd_Even, Connector_PinHeader_2.54mm:PinHeader_2x09_P2.54mm_Vertical, symbol Connector_Generic:Conn_02x09_Odd_Even
- added R364: DNP, Resistor_SMD:R_0805_2012Metric, symbol LiBCM-rescue:R
- HS1: footprint Linsight:Heatsink 573300D00010G -> Linsight:Heatsin-DV-T263-301E-TR
Connections:
- net +5V: now also C153.1
- net BATTSCI_DE: now also J4.3 (Pin_3)
- net BATTSCI_REn: now also J4.4 (Pin_4)
- net BUZZER: now also J4.7 (Pin_7)
- net COVER_SWITCH: now also J4.6 (Pin_6)
- net GND_ENG: now also C153.2, J4.1 (Pin_1), J4.17 (Pin_17), J4.18 (Pin_18), R364.1
- net GPIO-0: now also J4.5 (Pin_5)
- net GPIO-3: now also J4.8 (Pin_8)
- net LED3: now also J4.10 (Pin_10)
- net LED4: now also J4.12 (Pin_12)
- net SPI_CS_EXT: now also J4.9 (Pin_9)
- net SPI_CS_LTC: now also J4.15 (Pin_15)
- net SPI_MISO: now also J4.14 (Pin_14)
- net SPI_MOSI: now also J4.13 (Pin_13)
- net SPI_SCK: now also J4.16 (Pin_16)
- net TEMP_EN: now also J4.11 (Pin_11)
- new net 38(HW_VER1): J4.2 (Pin_2), R364.2
Other:
- note added: "HW_VER1/0:\nFF: REVA/B/C\nFL: REVD\nLF: RESERVED\nLL: RESERVED\nF=FLOAT\nL=GND"
- note added: "THIS CIRCUIT ALLOWS\nLiBCM TO TURN ITSELF\nOFF UNTIL THE NEXT\nKEY ON EVENT (WHEN\nIMA BATTERY EMPTY)"
- note removed: "THIS CIRCUIT ALLOWS LiBCM\nTO TURN OFF ENTIRE 5V RAIL\n(INCLUDING ITSELF) UNTIL\nTHE NEXT KEY ON EVENT.\n\nINTENDED USE: PREVENT DRAIN\nON DISCHARGED IMA BATTERY."
- moved on the sheet: BZ1, C11, C14, C143, C156, C157, C158, C159, C160, C17, C179, C18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
