File: Electronics/PCB (KiCAD)/RevD/KiCAD/LiBCM.kicad_pcb (KiCad board)
At the start: 4 copper layers, 355 x 160 mm, 715 parts, among them J1 Conn_01x08, J10 Screw_Terminal_01x01, J11 Screw_Terminal_01x08, J12 Conn_02x02, J13 Conn_01x20, J14 Conn_01x04, J15 Conn_01x02, J16 Conn_01x20, J17 Conn_01x14, J18 Conn_01x14, J19 Conn_02x02, J2 Conn_01x08, J20 Conn_02x02, J21 Conn_01x04, J22 Conn_01x08, J3 Conn_01x08, J4 Conn_02x08_Odd_Even, J5 Conn_01x08, J6 Conn_01x08, J7 Conn_01x08, J8 Conn_01x04, J9 Screw_Terminal_01x08, M1 Fan, M2 Fan, M3 Fan, P1 OEM_BCM_Connector, P2 Conn_WallPlug_Earth, Q1 Q_NMOS_GSD, Q10 Q_PMOS_GSD, Q11 Q_PMOS_GSD, Q12 Q_PMOS_GSD, Q13 Q_PMOS_GSD, Q14 Q_PMOS_GSD, Q15 Q_PMOS_GSD, Q16 Q_PMOS_GSD, Q17 Q_PMOS_GSD, Q18 Q_PMOS_GSD, Q19 Q_PMOS_GSD, Q2 Q_NMOS_GSD, Q20 Q_NPN_BCEC, Q21 Q_PMOS_GSD, Q22 Q_PMOS_GSD, Q23 Q_PMOS_GSD, Q24 Q_PMOS_GSD, Q25 Q_PMOS_GSD, Q26 Q_PMOS_GSD, Q27 Q_PMOS_GSD, Q28 Q_PMOS_GSD, Q29 Q_PMOS_GSD, Q3 Q_NMOS_GSD, Q30 Q_PMOS_GSD, Q31 Q_PMOS_GSD, Q32 Q_PMOS_GSD, Q33 Q_NPN_BCEC, Q34 Q_PMOS_GSD, Q35 Q_PMOS_GSD, Q36 Q_PMOS_GSD, Q37 Q_PMOS_GSD, Q38 Q_PMOS_GSD, Q39 Q_PMOS_GSD, Q4 Q_NMOS_GSD, Q40 Q_PMOS_GSD, Q41 Q_PMOS_GSD, Q42 Q_PMOS_GSD, Q43 Q_PMOS_GSD, Q44 Q_PMOS_GSD, Q45 Q_PMOS_GSD, Q46 Q_NPN_BCEC, Q47 Q_PMOS_GSD, Q48 Q_PMOS_GSD, Q49 Q_PMOS_GSD, Q5 Q_NMOS_GSD, Q50 Q_PMOS_GSD, Q51 Q_PMOS_GSD, Q52 Q_PMOS_GSD, Q53 Q_PMOS_GSD, Q54 Q_PMOS_GSD, Q55 Q_PMOS_GSD, Q56 Q_PMOS_GSD, Q57 Q_PMOS_GSD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

Commit message: RevD PCB Layout
Routing:
- net HVDC_POS_FUSED: track 184.9 -> 186.5 mm, vias 2 -> 8
- net /GRID_HVDC+: vias 0 -> 6
- added copper zone on B.Cu, net /GRID_HVDC+
- added copper zone on F.Cu, net /GRID_HVDC+
- added copper zone on B.Cu, net HVDC_POS_FUSED
- added copper zone on F.Cu, net HVDC_POS_FUSED

Commit message: Finished RevD PCB (except for possible HVAC switch change)
Parts:
- added C153: 22u, Capacitor_SMD:C_1210_3225Metric, F.Cu at (284.8, 87.3)
- added R364: DNP, Resistor_SMD:R_0805_2012Metric, F.Cu at (125.5, 150.0)
- HS1: footprint Linsight:Heatsink 573300D00010G -> Linsight:Heatsin-DV-T263-301E-TR
- J4: value Conn_02x08_Odd_Even -> Conn_02x09_Odd_Even; footprint Connector_PinHeader_2.54mm:PinHeader_2x08_P2.54mm_Vertical -> Connector_PinHeader_2.54mm:PinHeader_2x09_P2.54mm_Vertical
- moved D18 50.8 mm to (320.5, 40.8)
- moved C20 16.6 mm to (286.2, 79.0), turned to 270 degrees
- moved R76 15.0 mm to (279.5, 74.0)
- moved R60 14.2 mm to (304.8, 64.0)
- moved C24 14.0 mm to (302.2, 64.0)
- moved Q80 13.6 mm to (296.2, 82.2)
- moved U6 13.4 mm to (304.5, 56.0)
- moved R63 12.5 mm to (308.8, 59.8)
- moved R332 10.7 mm to (311.0, 57.5)
- moved C28 10.4 mm to (303.5, 72.8), turned to 0 degrees
- moved C180 10.3 mm to (276.0, 73.2), turned to 180 degrees
- moved R331 9.09 mm to (304.8, 104.2)
- moved D13 8.55 mm to (273.9, 80.0), turned to 180 degrees
- moved R61 8.55 mm to (308.8, 56.0), turned to 270 degrees
- moved U7 8.44 mm to (318.0, 53.0), turned to 0 degrees
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Connections:
- J4 pad 1: /BATTSCI_DE -> GND_ENG
- J4 pad 10: /LED4 -> /LED3
- J4 pad 11: /SPI_MOSI -> /TEMP_EN
- J4 pad 12: /SPI_MISO -> /LED4
- J4 pad 13: /SPI_CS_LTC -> /SPI_MOSI
- J4 pad 14: /SPI_SCK -> /SPI_MISO
- J4 pad 15: GND_ENG -> /SPI_CS_LTC
- J4 pad 16: GND_ENG -> /SPI_SCK
- J4 pad 2: /BATTSCI_REn -> /38(HW_VER1)
- J4 pad 3: /GPIO-0 -> /BATTSCI_DE
- J4 pad 4: /COVER_SWITCH -> /BATTSCI_REn
- J4 pad 5: /BUZZER -> /GPIO-0
- J4 pad 6: /GPIO-3 -> /COVER_SWITCH
- J4 pad 7: /SPI_CS_EXT -> /BUZZER
- J4 pad 8: /LED3 -> /GPIO-3
- J4 pad 9: /TEMP_EN -> /SPI_CS_EXT
Routing:
- net GND_ENG: track 3190.7 -> 3575.9 mm, vias 549 -> 624
- net +5V: track 767.6 -> 832.4 mm, vias 22 -> 26
- net HVDC_POS_FUSED: track 186.5 -> 233.8 mm, vias 8 -> 15
- net +15V: track 187.0 -> 220.6 mm, vias 1 -> 4
- net GND_CHASSIS: track 94.4 -> 74.7 mm
- net /L1: track 153.1 -> 136.0 mm, vias 17 -> 39
- net /GRID_SENSE: track 241.6 -> 225.6 mm
- net /38(HW_VER1): track 0.00 -> 12.3 mm
- net /GRID_PWM+: track 15.5 -> 4.47 mm
- net /+12V_FAN: track 35.3 -> 44.7 mm
- net /5V_SW_ALT: track 0.00 -> 9.31 mm
- net /GRID_PWM: track 248.9 -> 239.9 mm
- net /BATTSCI1: track 196.2 -> 203.5 mm
- net /I_SENSOR_POS: track 20.5 -> 13.8 mm
- net /5V_FB_ALT: track 0.00 -> 6.68 mm
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- added copper zone on F.Cu, net /+12V_FAN
- added copper zone on F.Cu, net /FAN-
- added copper zone on F.Cu, net /L1_GRID
- added copper zone on F.Cu, net /VDROP_13
- added copper zone on F.Cu, net /VDROP_14
Other:
- board text added: "6.3A@300VDC"
- board text added: "DANGER HVDC!"
- board text added: "HIGH VOLTAGE"
- board text added: "HVDC WHEN IMA SWITCH ON OR GRID CHARGER POWERED"
- board text added: "PRESENT EVEN"
- board text added: "SHORT THE FOLLOWING: 60S(IMA BATT): NONE 54S(IMA BATT): 60+ TO 54+ 4S(12V BATT): 60+ TO 52+ 3S(12V BATT): 60+ TO 51+"
- board text added: "TO USE LiDisplay: -J14: CONNECT CABLE -J15: REMOVE JUMPER TO USE HLINE: -J14: SHORT TX & RX -J15: SHORT PINS -P1: CONNECT HLINE TO BCM CONN B01"
- board text added: "WHEN IMA SWITCH OFF"
- board text removed: "54S IMA BATTERY: SHORT 60+ TO 54+ SHORT 49- TO 48+ LITHIUM 12V BATTERY: SHORT 60+ TO 52+ LEAVE 49- FLOATING!"
- board text removed: "8A@300VDC"
- board text removed: "CONNECTOR"
- board text removed: "DANGER! HVAC!!"
- board text removed: "DANGER: HVDC WHEN IMA SWITCH ON OR GRID CHARGER POWERED"
- board text removed: "IMA SWITCH IS OFF"
- board text removed: "PRESENT EVEN WHEN"
- board text removed: "TO USE HLINE: -J14: SHORT TX & RX -J15: SHORT PINS -P1: CONNECT HLINE TO BCM CONN B01 TO USE LiDisplay: -J14: CONNECT CABLE -J15: REMOVE JUMPER"

Commit message: Final RevD PCB
Parts:
- moved R74 0.25 mm to (302.2, 42.2)
- moved R75 0.25 mm to (302.2, 39.5)
- moved R77 0.25 mm to (302.5, 48.5)
- moved R79 0.25 mm to (302.5, 45.8)
Routing:
- net /L1: track 136.0 -> 165.6 mm, vias 39 -> 38
- net /TRIAC_GATE: track 36.0 -> 34.1 mm
- net /L1_UNFUSED: track 7.41 -> 8.66 mm
- net HVDC_NEG: track 179.2 -> 178.5 mm
- net GND_ISO_C: vias 7 -> 8
- added copper zone on B.Cu, net /L1_UNFUSED
- added copper zone on F.Cu, net /L1_UNFUSED
- added copper zone on F.Cu, net /LiBCM BMS/VREG_C
