File: Electronics/Lithium Batteries/5 Ah '5AhG3' Modules/PCB - Battery Heater/5AhG3 - 12S/RevB/KiCAD/5AhG3-12S.kicad_pcb (KiCad board)
At the start: 2 copper layers, 240.5 x 124 mm, 130 parts, among them J1 Screw_Terminal_01x02, J2 Screw_Terminal_01x02, J3 Screw_Terminal_01x03, J4 Screw_Terminal_01x03, J5 Conn_01x02, Q1 Q_NMOS_GDS, U1 APV1121S

Commit message: RevB Heater PCBs, Daughterboard Schematic
Parts:
- removed REF**: OSHW-Logo2_24.3x20mm_SilkScreen, Symbol:OSHW-Logo2_24.3x20mm_SilkScreen
- J3, J4: value Screw_Terminal_01x03 -> Screw_Terminal_01x02; footprint Connector_Phoenix_MC:PhoenixContact_MCV_1,5_3-G-3.5_1x03_P3.50mm_Vertical -> Connector_Phoenix_MC:PhoenixContact_MCV_1,5_2-G-3.5_1x02_P3.50mm_Vertical
- moved J1 15.2 mm to (308.5, 92.5)
- moved R111 15.0 mm to (295.5, 88.5), turned to 270 degrees
- moved R109 11.0 mm to (310.0, 83.2), turned to 180 degrees
- moved U1 10.3 mm to (302.5, 88.8), turned to 180 degrees
- moved R110 8.25 mm to (310.0, 80.8), turned to 180 degrees
- moved D1 5.59 mm to (302.0, 83.5), turned to 180 degrees
- moved J4 3.50 mm to (299.0, 113.0)
- moved R112 2.26 mm to (302.0, 80.8), turned to 180 degrees
Routing:
- net /GND_SAFE: track 25.3 -> 4.28 mm
- net /GPIO_L1: track 5.00 -> 8.67 mm
- net /GPIO: track 8.10 -> 11.6 mm
- net /HVDC_NEG_SWITCHED: track 352.9 -> 350.8 mm
- net /LEDn: track 2.81 -> 4.85 mm
- net /HVDC_NEG: track 67.0 -> 65.6 mm
- net /Q1_GATE: track 66.9 -> 65.6 mm
Other:
- outline, holes or cut-outs redrawn
- board text added: "300 VDC"
- board text added: "DANGER: HIGH VOLTAGE"
- board text added: "GPIO GND"
- board text added: "HEAT+ HEAT+ HVDC+ HVDC- HEAT- HEAT-"
- board text added: "TEMP"
- board text added: "WHEN WIRES CONNECTED!"
- board text removed: "300VDC"
- board text removed: "CONNECTOR"
- board text removed: "GND GPIO"
- board text removed: "HEAT+ HEAT+ HEAT+ HVDC+ HVDC- HEAT- HEAT- HEAT-"
- board text removed: "HIGH VOLTAGE! DANGER!"
- board text removed: "LINE MUST BE VISIBLE!"
- board text removed: "METAL HOLE THIS SIDE"
