File: Electronics/Lithium Batteries/5 Ah '5AhG3' Modules/PCB - Battery Heater/5AhG3 - 18S/RevB/KiCAD/5AhG3-18S.kicad_pcb (KiCad board)
At the start: 2 copper layers, 296.5 x 124 mm, 181 parts, among them J1 Conn_01x02

Commit message: RevB Heater PCBs, Daughterboard Schematic
Parts:
- removed R163, R164, R165, R166, R167, R168, R169, R170: 2k2, Resistor_SMD:R_2010_5025Metric
- added J2: Conn_01x02, Connector_PinHeader_2.54mm:PinHeader_1x02_P2.54mm_Horizontal, B.Cu at (359.8, 155.5)
- moved R157 2.12 mm to (345.5, 131.5), turned to 270 degrees
- moved R159 2.12 mm to (345.5, 140.5), turned to 270 degrees
- moved R155 0.25 mm to (347.0, 118.2)
Routing:
- net /HVDC_POS: track 401.5 -> 451.1 mm
- net Net-(R157-Pad2): track 44.4 -> 4.38 mm
- net /HVDC_NEG: track 399.3 -> 407.8 mm
- net Net-(R169-Pad2): track 6.00 -> 0.00 mm
- net Net-(R168-Pad2): track 6.00 -> 0.00 mm
- net Net-(R167-Pad2): track 6.00 -> 0.00 mm
- net Net-(R165-Pad2): track 6.00 -> 0.00 mm
- net Net-(R164-Pad2): track 6.00 -> 0.00 mm
- net Net-(R163-Pad2): track 6.00 -> 0.00 mm
- removed copper zone on B.Cu, net Net-(R163-Pad2)
- removed copper zone on B.Cu, net Net-(R164-Pad2)
- removed copper zone on B.Cu, net Net-(R165-Pad2)
- removed copper zone on B.Cu, net Net-(R167-Pad2)
- removed copper zone on B.Cu, net Net-(R168-Pad2)
- removed copper zone on B.Cu, net Net-(R169-Pad2)
Other:
- board text added: "HIGH VOLTAGE INTERCONNECT"
- board text added: "HVDC_A HVDC_B"
- board text removed: "LINE MUST BE VISIBLE!"
- board text removed: "METAL HOLE THIS SIDE"
