File: Electronics/PCB (KiCAD)/Daughterboard/RevA/KiCAD/LiBCM-Daughterboard/LiBCM-Daughterboard.kicad_pcb (KiCad board)
At the start: 4 copper layers, 166.8 x 78.2 mm, 61 parts, among them J1 Conn_01x03, J10 Conn_01x04, J11 Conn_01x04, J12 Conn_01x02, J13 Conn_01x04, J2 Conn_01x04, J3 Conn_01x07, J4 Conn_01x07, J5 Conn_02x03_Odd_Even, J6 Conn_01x04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

Commit message: As Ordered Daughterboard
Parts:
- J6, J7, J9: moved to B.Cu
- moved C1 0.20 mm to (121.5, 150.5)
- turned J6 to 270 degrees
- turned J7 to 90 degrees
- turned J9 to 90 degrees
Routing:
- net /GRID_POS: track 19.0 -> 38.4 mm
- net /HEAT_NEG: track 21.7 -> 38.7 mm, vias 0 -> 1
- net GNDPWR: track 76.6 -> 85.0 mm, vias 6 -> 11
- net GND: track 276.0 -> 283.4 mm, vias 7 -> 27
- net /HVDC_5V_REF: track 74.7 -> 82.0 mm
- net /MISO: track 64.8 -> 61.9 mm
- net /MOSI: track 74.3 -> 71.8 mm
- net /FLASH_CS: track 28.7 -> 30.0 mm
- net +5V: track 131.0 -> 131.8 mm
- added copper zone on B.Cu, net +5V
- added copper zone on F.Cu, net +5V
- added copper zone on B.Cu, net /GRID_POS
- added copper zone on B.Cu, net /HVDC_POS_AUX
- added copper zone on F.Cu, net /HVDC_POS_AUX
- added copper zone on B.Cu, net /HVDC_POS_BATT
- added copper zone on B.Cu, net GND
- added copper zone on F.Cu, net GND
- added copper zone on B.Cu, net GNDPWR
Other:
- board size 166.8 x 78.2 mm -> 166.8 x 30 mm
- board text added: "+5V"
- board text added: "1500 W CHARGER"
- board text added: "47Ah HEATER"
- board text added: "4x20 LCD"
- board text added: "ADAFRUIT#4899"
- board text added: "CAN"
- board text added: "CHONKER HEAT SINK MOUNTS"
- board text added: "CS MOSI MISO SCK GND N/C VCC"
- board text added: "DESIGNED BY IC.NET USER 'MUDDER' (A.K.A. JOHN SULLIVAN) LINSIGHT.ORG"
- board text added: "FAN TACHOMETER"
- board text added: "FLASH"
- board text added: "FUSE: HEATER"
- board text added: "FUSE:GRID CHARGER"
- board text added: "GND"
- board text added: "GND SDA SCL 5V"
- board text added: "GRID CHARGER BLOCKING DIODE"
- board text added: "GRID CURRENT LIMIT"
- board text added: "HEAT ISO"
- board text added: "HEATER SWITCH"
- board text added: "LiCONTROL"
- board text added: "MCP2515"
- board text added: "MEMORY IS THE MOTHER OF ALL WISDOM"
- board text added: "POWER IS NOTHING WITHOUT CONTROL"
- board text added: "Q: "WHEN WILL LiBCM EXIT BETA?" A: "WHEN IT'S READY" -BULL DOG"
- board text added: "TO GRID CHARGER CONTROL"
- board text added: "TO GRID CHARGER OUTPUT"
- board text added: "TO IMA JUNCTION BOARD"
- board text added: "TO LiBCM SCREW TERMINALS"
- board text added: "USE EITHER 4X20 OR MCP2515 (BUT NOT BOTH)"
- board text added: "USER SWITCH"
- board text added: "github.com/doppelhub/Honda_Insight_LiBCM/tree/main/Electronics/PCB%20(KiCAD)/Daughterboard"
- board text removed: "1500 W CHARGER BLOCKING DIODE"
