File: Electronics/PCB (KiCAD)/Daughterboard/RevB/KiCAD/LiBCM-Daughterboard/LiBCM-Daughterboard.kicad_pcb (KiCad board)
At the start: 4 copper layers, 166.8 x 31 mm, 75 parts, among them J10 Conn_01x04, J11 Conn_01x04, J12 Conn_01x02, J13 Conn_01x05, J2 Conn_01x04, J3 Conn_01x07, J4 Conn_01x07, J5 Conn_02x03_Odd_Even, J6 Conn_01x04, J7 Conn_01x08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

Commit message: Daughterboard: V2 RevB BOM, Pick&Place File
Parts:
- removed D2: LED, LED_SMD:LED_0805_2012Metric
- added R36: 100, Resistor_SMD:R_0805_2012Metric, F.Cu at (151.5, 135.8)
- R16, R18, R5: value 100k -> DNP
- R22: value 100 -> 20
- R28: value 71k5 -> 10k
- R30: value 100 -> 768
Connections:
- net /ILIM_DIV renamed /ILIM_LED_1
- R14 pad 1: /ILIM_LED2 -> /ILIM_LED_2
- U3 pad 2: /ILIM_LED -> /ILIM_LED_3
Routing:
- net /ILIM_LED_2: track 0.00 -> 4.01 mm
- net /ILIM_LED2: track 4.01 -> 0.00 mm
- net /ILIM_LED_3: track 0.00 -> 4.01 mm
- net /ILIM_LED: track 4.01 -> 0.00 mm
